File: hardware/EuroPi/kicad/EuroPi.kicad_sch (KiCad schematic)
At the start: 92 parts, among them IC1 TL074, IC2 TL074, IC3 MCP6002, J1 Thonkiconn_Mono_Jack, J2 Thonkiconn_Mono_Jack, J3 Thonkiconn_Mono_Jack, J4 Thonkiconn_Mono_Jack, J5 Thonkiconn_Mono_Jack, J6 Thonkiconn_Mono_Jack, J7 Thonkiconn_Mono_Jack, J8 Thonkiconn_Mono_Jack, Q1 2N2222, SW1 SW_Push, SW2 SW_Push

Commit message: save as kicad 7
Parts:
- D1, D2, D3, D4: value DIODE -> ${SIM.PARAMS}; Spice_Netlist_Enabled Y -> (none); Spice_Primitive D -> (none)

Commit message: fix resistor sides, routing
Parts:
- R13, R14, R15, R16, R17, R18: value 1K -> 4K7
Changed lines of the file:
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@@
       (effects (font (size 1.27 1.27)))
     )
-    (property "Value" "1K" (at 176.3014 53.34 90)
+    (property "Value" "4K7" (at 176.3014 53.34 90)
       (effects (font (size 1.27 1.27)))
     )
@@
       (effects (font (size 1.27 1.27)))
     )
-    (property "Value" "1K" (at 274.0914 53.34 90)
+    (property "Value" "4K7" (at 274.0914 53.34 90)
       (effects (font (size 1.27 1.27)))
     )
@@
       (effects (font (size 1.27 1.27)))
     )
-    (property "Value" "1K" (at 371.8814 53.34 90)
+    (property "Value" "4K7" (at 371.8814 53.34 90)
       (effects (font (size 1.27 1.27)))
     )
@@
       (effects (font (size 1.27 1.27)))
     )
-    (property "Value" "1K" (at 176.3014 109.22 90)
+    (property "Value" "4K7" (at 176.3014 109.22 90)
       (effects (font (size 1.27 1.27)))
     )
@@
       (effects (font (size 1.27 1.27)))
     )
-    (property "Value" "1K" (at 274.0914 109.22 90)
+    (property "Value" "4K7" (at 274.0914 109.22 90)
       (effects (font (size 1.27 1.27)))
     )
@@
       (effects (font (size 1.27 1.27)))
     )
-    (property "Value" "1K" (at 371.8814 109.22 90)
-      (effects (font (size 1.27 1.27)))
-    )
+    (property "Value" "4K7" (at 371.8814 109.22 90)
+      (effects (font (size 1.27 1.27)))
+    )

Commit message: kicad save
Connections:
- net EARTH J is gone; now on net Earth: C7.2, C8.2, CONN2.1 (Pin_1), CONN7.3 (Pin_3), J1.1 (E), J2.1 (E), J3.1 (E), J4.1 (E), J5.1 (E), J6.1 (E), J7.1 (E), J8.1 (E), LED1.1 (K), LED2.1 (K), LED3.1 (K), LED4.1 (K), LED5.1 (K), LED6.1 (K), SW1.1, SW2.1, VR1.3, VR2.3
Changed lines of the file:
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@@
+    )
+  )
+  (symbol (lib_id "power:Earth") (at 115.57 198.12 0) (unit 1)
+    (in_bom yes) (on_board yes) (dnp no)
+    (property "Reference" "#PWR02" (at 115.57 204.47 0)
+      (effects (font (size 1.27 1.27)) hide)
+    )
+    (property "Value" "Earth" (at 115.57 201.93 0)
+      (effects (font (size 1.27 1.27)) hide)
+    )
+    (property "Footprint" "" (at 115.57 198.12 0)
+      (effects (font (size 1.27 1.27)) hide)
+    )
+    (property "Datasheet" "~" (at 115.57 198.12 0)
+      (effects (font (size 1.27 1.27)) hide)
+    )
+    (pin "1")
+    (instances
+      (project "europi"
+        (path "/a8447faf-e0a0-4c4a-ae53-4d4b28669151"
+          (reference "#PWR02") (unit 1)
+        )
+      )
     )
   )
@@
         )
       )
+    )
+  )
+  (symbol (lib_id "power:Earth") (at 115.57 171.45 0) (unit 1)
+    (in_bom yes) (on_board yes) (dnp no)
+    (property "Reference" "#PWR01" (at 115.57 177.8 0)
+      (effects (font (size 1.27 1.27)) hide)
+    )
+    (property "Value" "Earth" (at 115.57 175.26 0)
+      (effects (font (size 1.27 1.27)) hide)
+    )
+    (property "Footprint" "" (at 115.57 171.45 0)
+      (effects (font (size 1.27 1.27)) hide)
+    )
+    (property "Datasheet" "~" (at 115.57 171.45 0)
+      (effects (font (size 1.27 1.27)) hide)
+    )
+    (pin "1")
+    (instances
+      (project "europi"
+        (path "/a8447faf-e0a0-4c4a-ae53-4d4b28669151"
+          (reference "#PWR01") (unit 1)
+        )
+      )
