File: hardware/EuroPi-X/kicad/EuroPi-X.kicad_pcb (KiCad board)
At the start: 2 copper layers, 40.6 x 110 mm, 53 parts, among them J1 USB_C_Receptacle_USB2.0, J3 Thonkiconn_Mono_Jack, J4 Thonkiconn_Mono_Jack, J5 Thonkiconn_Mono_Jack, J6 Thonkiconn_Mono_Jack, SW1 RESET, SW2 BOOT, U1 RP2040, Y1 Crystal_GND2

Commit message: kicad save
Parts:
- removed the J1 at (69.8, -10.2)
- removed the J3 at (5.20, 82.5)
- removed the J3 at (5.12, 101.6)
- removed the J4 at (15.2, 101.6)
- removed the J4 at (15.2, 63.5)
- removed the J4 at (15.3, 82.5)
- removed the J5 at (25.4, 101.6)
- removed the J5 at (25.3, 63.5)
- removed the J5 at (25.4, 82.5)
- removed the J6 at (35.5, 101.6)
- removed the J6 at (35.6, 82.5)
- removed the J6 at (35.4, 63.5)
- removed LED (x8): LED 3mm, Eurorack:LED 3mm
- removed POT (x2): Potentiometer 9mm Vertical Linear, Eurorack:Potentiometer 9mm Vertical Linear Centred
- removed SW (x2): Switch Tactile Momentary C&K, Eurorack:Switch Tactile Momentary C&K
- added C14: 1u, Capacitor_SMD:C_0402_1005Metric, F.Cu at (64.8, 61.3)
- added C15: 1u, Capacitor_SMD:C_0402_1005Metric, F.Cu at (67.6, 49.5)
- added C16: 100n, Capacitor_SMD:C_0402_1005Metric, F.Cu at (67.6, 51.4)
- added C17: 100n, Capacitor_SMD:C_0402_1005Metric, F.Cu at (67.6, 53.4)
- added C18: 100p, Capacitor_SMD:C_0402_1005Metric, F.Cu at (67.6, 55.4)
- added C19: 100p, Capacitor_SMD:C_0402_1005Metric, F.Cu at (67.6, 57.3)
- added C20: 100p, Capacitor_SMD:C_0402_1005Metric, F.Cu at (67.6, 59.3)
- added C21: 100p, Capacitor_SMD:C_0402_1005Metric, F.Cu at (67.6, 61.3)
- added C22: 100p, Capacitor_SMD:C_0402_1005Metric, F.Cu at (70.5, 49.5)
- added C23: 100p, Capacitor_SMD:C_0402_1005Metric, F.Cu at (70.5, 51.4)
- added C24: 1u, Capacitor_SMD:C_0402_1005Metric, F.Cu at (70.5, 53.4)
- added C25: 100n, Capacitor_SMD:C_0402_1005Metric, F.Cu at (70.5, 55.4)
- added D1: D, Diode_SMD:D_0402_1005Metric, F.Cu at (89.0, 60.9)
- added D2: D, Diode_SMD:D_0402_1005Metric, F.Cu at (89.0, 62.9)
- added DAC1: MCP4728, Package_SO:MSOP-10_3x3mm_P0.5mm, F.Cu at (81.6, 21.5)
- added DAC2: MCP4728, Package_SO:MSOP-10_3x3mm_P0.5mm, F.Cu at (81.6, 26.2)
- added J10: Thonkiconn_Mono_Jack, Eurorack:Thonkiconn Mono Jack, F.Cu at (15.2, 64.8)
- added J11: Thonkiconn_Mono_Jack, Eurorack:Thonkiconn Mono Jack, F.Cu at (25.4, 64.8)
- added J12: Thonkiconn_Mono_Jack, Eurorack:Thonkiconn Mono Jack, F.Cu at (35.6, 64.8)
- added J13: Conn_01x30_Pin, Connector_FFC-FPC:Hirose_FH41-30S-0.5SH_1x30_1MP_1SH_P0.5mm_Horizontal, F.Cu at (21.0, 19.7)
- added J2: Thonkiconn_Mono_Jack, Eurorack:Thonkiconn Mono Jack, F.Cu at (15.2, 83.2)
- added J3: Thonkiconn_Mono_Jack, Eurorack:Thonkiconn Mono Jack, F.Cu at (25.4, 83.2)
- added J4: Thonkiconn_Mono_Jack, Eurorack:Thonkiconn Mono Jack, F.Cu at (35.6, 83.2)
- added J5: Thonkiconn_Mono_Jack, Eurorack:Thonkiconn Mono Jack, F.Cu at (5.08, 101.6)
- added J6: Thonkiconn_Mono_Jack, Eurorack:Thonkiconn Mono Jack, F.Cu at (15.2, 101.6)
- added J7: Thonkiconn_Mono_Jack, Eurorack:Thonkiconn Mono Jack, F.Cu at (25.4, 101.6)
- added J8: Thonkiconn_Mono_Jack, Eurorack:Thonkiconn Mono Jack, F.Cu at (35.6, 101.6)
- added J9: Thonkiconn_Mono_Jack, Eurorack:Thonkiconn Mono Jack, F.Cu at (5.08, 64.8)
- added JUMPER1: UNI/BIPOLAR, Connector_PinHeader_2.54mm:PinHeader_1x03_P2.54mm_Vertical, F.Cu at (87.8, 39.3)
- added LED1: SK6805, LED_SMD:LED_SK6805_PLCC4_2.4x2.7mm_P1.3mm, F.Cu at (5.08, 74.9)
- added LED10: SK6805, LED_SMD:LED_SK6805_PLCC4_2.4x2.7mm_P1.3mm, F.Cu at (15.2, 56.5)
- added LED11: SK6805, LED_SMD:LED_SK6805_PLCC4_2.4x2.7mm_P1.3mm, F.Cu at (25.4, 56.5)
- added LED12: SK6805, LED_SMD:LED_SK6805_PLCC4_2.4x2.7mm_P1.3mm, F.Cu at (35.6, 56.5)
- added LED2: SK6805, LED_SMD:LED_SK6805_PLCC4_2.4x2.7mm_P1.3mm, F.Cu at (15.2, 74.9)
- added LED3: SK6805, LED_SMD:LED_SK6805_PLCC4_2.4x2.7mm_P1.3mm, F.Cu at (25.4, 74.9)
- added LED4: SK6805, LED_SMD:LED_SK6805_PLCC4_2.4x2.7mm_P1.3mm, F.Cu at (35.6, 74.9)
- added LED5: SK6805, LED_SMD:LED_SK6805_PLCC4_2.4x2.7mm_P1.3mm, F.Cu at (5.08, 93.3)
- added LED6: SK6805, LED_SMD:LED_SK6805_PLCC4_2.4x2.7mm_P1.3mm, F.Cu at (15.2, 93.3)
- added LED7: SK6805, LED_SMD:LED_SK6805_PLCC4_2.4x2.7mm_P1.3mm, F.Cu at (25.4, 93.3)
- added LED8: SK6805, LED_SMD:LED_SK6805_PLCC4_2.4x2.7mm_P1.3mm, F.Cu at (35.6, 93.3)
- added LED9: SK6805, LED_SMD:LED_SK6805_PLCC4_2.4x2.7mm_P1.3mm, F.Cu at (5.08, 56.5)
- added P1: Potentiometer_9mm_Vertical_Linear, Eurorack:Potentiometer 9mm Vertical Linear Centred, F.Cu at (10.2, 30.5)
- added P2: Potentiometer_9mm_Vertical_Linear, Eurorack:Potentiometer 9mm Vertical Linear Centred, F.Cu at (30.5, 30.5)
- added R10: 1K, Resistor_SMD:R_0402_1005Metric, F.Cu at (52.7, 20.1)
- added R11: 100K, Resistor_SMD:R_0402_1005Metric, F.Cu at (52.7, 22.1)
- added R12: 100K, Resistor_SMD:R_0402_1005Metric, F.Cu at (52.7, 24.1)
- added R13: 100K, Resistor_SMD:R_0402_1005Metric, F.Cu at (52.7, 26.1)
- added R14: 100K, Resistor_SMD:R_0402_1005Metric, F.Cu at (52.7, 28.1)
- added R15: 270K, Resistor_SMD:R_0402_1005Metric, F.Cu at (52.7, 30.1)
- added R16: 270K, Resistor_SMD:R_0402_1005Metric, F.Cu at (52.7, 32.0)
- added R17: 1K, Resistor_SMD:R_0402_1005Metric, F.Cu at (52.7, 34.0)
- added R18: 1K, Resistor_SMD:R_0402_1005Metric, F.Cu at (52.7, 36.0)
- added R19: 27R4, Resistor_SMD:R_0402_1005Metric, F.Cu at (55.6, 20.1)
- added R20: 100K, Resistor_SMD:R_0402_1005Metric, F.Cu at (55.6, 22.1)
- added R21: 100K, Resistor_SMD:R_0402_1005Metric, F.Cu at (55.6, 24.1)
- added R22: 100K, Resistor_SMD:R_0402_1005Metric, F.Cu at (55.6, 26.1)
- added R23: 100K, Resistor_SMD:R_0402_1005Metric, F.Cu at (55.6, 28.1)
- added R24: 270K, Resistor_SMD:R_0402_1005Metric, F.Cu at (55.6, 30.1)
- added R25: 270K, Resistor_SMD:R_0402_1005Metric, F.Cu at (55.6, 32.0)
- added R26: 1K, Resistor_SMD:R_0402_1005Metric, F.Cu at (55.6, 34.0)
- added R27: 1K, Resistor_SMD:R_0402_1005Metric, F.Cu at (55.6, 36.0)
- added R28: 100K, Resistor_SMD:R_0402_1005Metric, F.Cu at (58.5, 20.1)
- added R29: 100K, Resistor_SMD:R_0402_1005Metric, F.Cu at (58.5, 22.1)
- added R30: 100K, Resistor_SMD:R_0402_1005Metric, F.Cu at (58.5, 24.1)
- added R31: 100K, Resistor_SMD:R_0402_1005Metric, F.Cu at (58.5, 26.1)
- added R32: 270K, Resistor_SMD:R_0402_1005Metric, F.Cu at (58.5, 28.1)
- added R33: 270K, Resistor_SMD:R_0402_1005Metric, F.Cu at (58.5, 30.1)
- added R34: 1K, Resistor_SMD:R_0402_1005Metric, F.Cu at (58.5, 32.0)
- added R35: 1K, Resistor_SMD:R_0402_1005Metric, F.Cu at (58.5, 34.0)
- added R36: 100K, Resistor_SMD:R_0402_1005Metric, F.Cu at (58.5, 36.0)
- added R37: 100K, Resistor_SMD:R_0402_1005Metric, F.Cu at (61.4, 20.1)
- added R38: 100K, Resistor_SMD:R_0402_1005Metric, F.Cu at (61.4, 22.1)
- added R39: 100K, Resistor_SMD:R_0402_1005Metric, F.Cu at (61.4, 24.1)
- added R40: 270K, Resistor_SMD:R_0402_1005Metric, F.Cu at (61.4, 26.1)
- added R41: 270K, Resistor_SMD:R_0402_1005Metric, F.Cu at (61.4, 28.1)
- added R42: 1K, Resistor_SMD:R_0402_1005Metric, F.Cu at (61.4, 30.1)
- added R43: 1K, Resistor_SMD:R_0402_1005Metric, F.Cu at (61.4, 32.0)
- added R44: 100K, Resistor_SMD:R_0402_1005Metric, F.Cu at (61.4, 34.0)
- added R45: 15K, Resistor_SMD:R_0402_1005Metric, F.Cu at (61.4, 36.0)
- added R46: 2K2, Resistor_SMD:R_0402_1005Metric, F.Cu at (64.3, 20.1)
- added R47: 10K, Resistor_SMD:R_0402_1005Metric, F.Cu at (64.3, 22.1)
- added R48: 100K, Resistor_SMD:R_0402_1005Metric, F.Cu at (64.3, 24.1)
- added R49: 10K, Resistor_SMD:R_0402_1005Metric, F.Cu at (64.3, 26.1)
- added R50: 100K, Resistor_SMD:R_0402_1005Metric, F.Cu at (64.3, 28.1)
- added R51: 100K, Resistor_SMD:R_0402_1005Metric, F.Cu at (64.3, 30.1)
- added R52: 15K, Resistor_SMD:R_0402_1005Metric, F.Cu at (64.3, 32.0)
- added R53: 10K, Resistor_SMD:R_0402_1005Metric, F.Cu at (64.3, 34.0)
- added R54: 100K, Resistor_SMD:R_0402_1005Metric, F.Cu at (64.3, 36.0)
- added R55: 100K, Resistor_SMD:R_0402_1005Metric, F.Cu at (67.2, 20.1)
- added R56: 15K, Resistor_SMD:R_0402_1005Metric, F.Cu at (67.2, 22.1)
- added R57: 10K, Resistor_SMD:R_0402_1005Metric, F.Cu at (67.2, 24.1)
- added R58: 100K, Resistor_SMD:R_0402_1005Metric, F.Cu at (67.2, 26.1)
- added R59: 100K, Resistor_SMD:R_0402_1005Metric, F.Cu at (67.2, 28.1)
- added R60: 15K, Resistor_SMD:R_0402_1005Metric, F.Cu at (67.2, 30.1)
- added R61: ~, Resistor_SMD:R_0402_1005Metric, F.Cu at (67.2, 32.0)
- added R9: 10K, Resistor_SMD:R_0402_1005Metric, F.Cu at (49.8, 36.0)
- added SW3: BOOT, Button_Switch_THT:SW_PUSH_6mm_H4.3mm, F.Cu at (80.2, 51.7)
- added U11: LM4040DBZ-10, Package_TO_SOT_SMD:SOT-23, F.Cu at (87.8, 25.8)
- added U4: ~, Package_TO_SOT_SMD:TO-252-3_TabPin4, F.Cu at (55.2, 52.5)
- added U5: ~, Package_TO_SOT_SMD:TO-252-3_TabPin4, F.Cu at (55.2, 60.5)
- added U6: TL074, Package_SO:SOIC-16_3.9x9.9mm_P1.27mm, F.Cu at (52.5, 42.7)
- added U7: TL074, Package_SO:SOIC-16_3.9x9.9mm_P1.27mm, F.Cu at (61.0, 42.7)
- added U7: TL074, Package_SO:SOIC-16_3.9x9.9mm_P1.27mm, F.Cu at (69.4, 42.7)
- added U8: MCP3428, Package_SO:SOIC-14_3.9x8.7mm_P1.27mm, F.Cu at (86.4, 54.8)
- added U9: MCP6004, Package_SO:TSSOP-14_4.4x5mm_P0.65mm, F.Cu at (73.1, 31.7)
- added USB1: USB_C_Receptacle_USB2.0, Connector_USB:USB_C_Receptacle_Amphenol_12401548E4-2A, F.Cu at (79.6, 43.3)
- C10, C11: value 100n -> 100p
- C12, C13: value 10p -> 100n
- C2, C3, C6: value 100n -> 1u
- C4, C5: value 1u -> 100n
- C7: value 100n -> 10p
- C8: value 1u -> 10p
- R1, R2: value 27R4 -> 2K2
- R3, R4: value 5K1 -> 27R4
- R5, R6: value 10K -> 5K1
- R7: value 27R4 -> 10K
- R8: value 1K -> 10K
- SW1: value RESET -> BOOT; footprint Button_Switch_SMD:SW_SP3T_PCM13 -> Eurorack:Switch Tactile Momentary C&K
- SW2: footprint Button_Switch_SMD:SW_SP3T_PCM13 -> Eurorack:Switch Tactile Momentary C&K
- U1: value RP2040 -> LM4030-4.096; footprint Package_DFN_QFN:QFN-56-1EP_7x7mm_P0.4mm_EP3.2x3.2mm -> Package_TO_SOT_SMD:SOT-23-5
- U2: value ~ -> LM4040DBZ-2.0; footprint Package_TO_SOT_SMD:TO-252-3_TabPin4 -> Package_TO_SOT_SMD:SOT-23
- U3: value ~ -> RP2040; footprint Package_TO_SOT_SMD:TO-252-3_TabPin4 -> Package_DFN_QFN:QFN-56-1EP_7x7mm_P0.4mm_EP3.2x3.2mm
- moved SW1 115.0 mm to (7.62, 50.8)
- moved SW2 94.4 mm to (27.9, 50.8)
- moved C6 90.6 mm to (61.9, 59.3)
- moved C7 90.6 mm to (61.9, 61.3)
- moved C11 87.4 mm to (64.8, 55.4)
- moved C12 87.4 mm to (64.8, 57.3)
- moved C13 87.4 mm to (64.8, 59.3)
- moved C1 81.0 mm to (61.9, 49.5)
- moved C2 81.0 mm to (61.9, 51.4)
- moved C3 81.0 mm to (61.9, 53.4)
- moved C4 81.0 mm to (61.9, 55.4)
- moved C5 81.0 mm to (61.9, 57.3)
- moved C10 77.9 mm to (64.8, 53.4)
- moved C8 77.9 mm to (64.8, 49.5)
- moved C9 77.9 mm to (64.8, 51.4)
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- renumbered J3 to J1
Connections:
- C1 pad 1: Net-(U1-VREG_VOUT) -> Net-(U3-VREG_VOUT)
- C10 pad 1: IOVDD -> Net-(U6A-+)
- C10 pad 2: Earth -> Net-(C10-Pad2)
- C11 pad 1: IOVDD -> Net-(U7A-+)
- C11 pad 2: Earth -> Net-(C11-Pad2)
- C12 pad 1: Earth -> ADC_AVDD
- C12 pad 2: XTAL_IN -> Earth
- C13 pad 1: Earth -> IOVDD
- C13 pad 2: XTAL_OUT -> Earth
- C2 pad 1: Net-(U1-VREG_VOUT) -> /-4.096VREF
- C3 pad 1: Net-(U1-VREG_VOUT) -> /-2.048VREF
- C4 pad 1: +5V -> Net-(U3-VREG_VOUT)
- C5 pad 1: IOVDD -> Net-(U3-VREG_VOUT)
- C6 pad 1: ADC_AVDD -> +5V
- C7 pad 1: IOVDD -> Earth
- C7 pad 2: Earth -> XTAL_IN
- C8 pad 1: ADC_AVDD -> Earth
- C8 pad 2: Earth -> XTAL_OUT
- J1 pad 1: unconnected-(J3-E-Pad1) -> Earth
- J1 pad 3: unconnected-(J3-T-Pad3) -> Net-(J1-T)
- R1 pad 1: USB_DP -> /-4.096VREF
- R1 pad 2: Net-(U1-USB_DP) -> -12V
- R2 pad 1: USB_DM -> /-2.048VREF
- R2 pad 2: Net-(U1-USB_DM) -> -12V
- R3 pad 1: Net-(J1-CC1) -> USB_DP
- R3 pad 2: Earth -> Net-(U3-USB_DP)
- R4 pad 1: Net-(J1-CC2) -> USB_DM
- R4 pad 2: Earth -> Net-(U3-USB_DM)
- R5 pad 1: RUN -> Net-(USB1-CC1)
- R5 pad 2: IOVDD -> Earth
- R6 pad 1: IOVDD -> Net-(USB1-CC2)
- R6 pad 2: QSPI_CS -> Earth
- R7 pad 1: IOVDD -> /OUTPUT_MODE
- R7 pad 2: ADC_AVDD -> /DAC_OFFSET
- R8 pad 1: QSPI_CS -> Earth
- R8 pad 2: Net-(R8-Pad2) -> /OUTPUT_MODE
- SW1 pad 1: RUN -> /BUTTON_1
- SW2 pad 1: Net-(R8-Pad2) -> /BUTTON_2
- U1 pad 1: IOVDD -> (no net)
- U1 pad 2: unconnected-(U1-GPIO0-Pad2) -> (no net)
- U1 pad 3: unconnected-(U1-GPIO1-Pad3) -> (no net)
- U1 pad 4: unconnected-(U1-GPIO2-Pad4) -> Earth
- U1 pad 5: unconnected-(U1-GPIO3-Pad5) -> /-4.096VREF
- U2 pad 1: IOVDD -> Earth
- U2 pad 2: Earth -> /-2.048VREF
- U2 pad 3: +5V -> (no net)
- U3 pad 1: QSPI_CS -> IOVDD
- U3 pad 2: QSPI_SD1 -> IOVDD
- U3 pad 3: QSPI_SD2 -> Earth
- U3 pad 4: Earth -> /OUTPUT_MODE

Commit message: kicad save and pdf schematic
Parts:
- added C26: 100n, Capacitor_SMD:C_0402_1005Metric, F.Cu at (123.6, 53.9)
- added C27: 100n, Capacitor_SMD:C_0402_1005Metric, F.Cu at (123.6, 55.9)
- added C28: 100n, Capacitor_SMD:C_0402_1005Metric, F.Cu at (123.6, 57.9)
- added C29: 100n, Capacitor_SMD:C_0402_1005Metric, F.Cu at (123.6, 59.8)
- added C30: 100n, Capacitor_SMD:C_0402_1005Metric, F.Cu at (123.6, 61.8)
- added J14: Conn_02x12_Counter_Clockwise, Connector_PinSocket_2.54mm:PinSocket_2x12_P2.54mm_Vertical, F.Cu at (81.3, 8.89)
- added J15: Conn_02x12_Counter_Clockwise, Connector_PinHeader_2.54mm:PinHeader_2x12_P2.54mm_Vertical, B.Cu at (34.3, 8.89)
- moved R47 74.1 mm to (8.26, 70.5)
- moved U9 68.2 mm to (137.5, 53.9), turned to 90 degrees
- moved U4 66.3 mm to (120.5, 40.9)
- moved U5 66.3 mm to (120.5, 48.9)
- moved R49 63.9 mm to (18.4, 70.5)
- moved C25 58.9 mm to (27.9, 14.6)
- moved R10 57.3 mm to (97.5, 55.7)
- moved R11 57.3 mm to (97.5, 57.7)
- moved Y1 57.1 mm to (130.5, 63.4)
- moved DAC1 56.9 mm to (138.2, 27.8)
- moved DAC2 56.9 mm to (138.2, 32.5)
- moved R55 56.4 mm to (109.2, 57.7)
- moved R19 54.9 mm to (100.5, 51.8)
- moved R20 54.9 mm to (100.5, 53.7)
- moved R21 54.9 mm to (100.5, 55.7)
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Connections:
- C25 pad 2: Earth -> /GND_FRONT
- J1 pad 1: Earth -> /GND_FRONT
- J1 pad 3: Net-(J1-T) -> /CV_OUTPUT_1_FRONT
- J10 pad 1: Earth -> /GND_FRONT
- J10 pad 3: Net-(J10-T) -> /CV_INPUT_2_FRONT
- J11 pad 1: Earth -> /GND_FRONT
- J11 pad 3: Net-(J11-T) -> /CV_INPUT_3_FRONT
- J12 pad 1: Earth -> /GND_FRONT
- J12 pad 3: Net-(J12-T) -> /CV_INPUT_4_FRONT
- J13 pad 10: IOVDD -> /+3.3V_FRONT
- J13 pad 11: Earth -> /GND_FRONT
- J13 pad 12: Earth -> /GND_FRONT
- J13 pad 13: Earth -> /GND_FRONT
- J13 pad 14: IOVDD -> /+3.3V_FRONT
- J13 pad 15: /D/C# -> /OLED_D/C_FRONT
- J13 pad 16: Earth -> /GND_FRONT
- J13 pad 17: Earth -> /GND_FRONT
- J13 pad 18: /D0 -> /OLED_CLK_FRONT
- J13 pad 19: /D1 -> /OLED_DIN_FRONT
- J13 pad 21: Earth -> /GND_FRONT
- J13 pad 22: Earth -> /GND_FRONT
- J13 pad 23: Earth -> /GND_FRONT
- J13 pad 24: Earth -> /GND_FRONT
- J13 pad 25: Earth -> /GND_FRONT
- J13 pad 28: IOVDD -> /+3.3V_FRONT
- J13 pad 29: Earth -> /GND_FRONT
- J13 pad 6: IOVDD -> /+3.3V_FRONT
- J13 pad 8: Earth -> /GND_FRONT
- J13 pad 9: IOVDD -> /+3.3V_FRONT
- J2 pad 1: Earth -> /GND_FRONT
- J2 pad 3: Net-(J2-T) -> /CV_OUTPUT_5_FRONT
- J3 pad 1: Earth -> /GND_FRONT
- J3 pad 3: Net-(J3-T) -> /CV_OUTPUT_2_FRONT
- J4 pad 1: Earth -> /GND_FRONT
- J4 pad 3: Net-(J4-T) -> /CV_OUTPUT_6_FRONT
- J5 pad 1: Earth -> /GND_FRONT
- J5 pad 3: Net-(J5-T) -> /CV_OUTPUT_3_FRONT
- J6 pad 1: Earth -> /GND_FRONT
- J6 pad 3: Net-(J6-T) -> /CV_OUTPUT_7_FRONT
- J7 pad 1: Earth -> /GND_FRONT
- J7 pad 3: Net-(J7-T) -> /CV_OUTPUT_4_FRONT
- J8 pad 1: Earth -> /GND_FRONT
- J8 pad 3: Net-(J8-T) -> /CV_OUTPUT_8_FRONT
- J9 pad 1: Earth -> /GND_FRONT
- J9 pad 3: Net-(J9-T) -> /CV_INPUT_1_FRONT
- LED1 pad 2: Earth -> /GND_FRONT
- LED1 pad 3: /NEOPIXEL_DATA -> /NEOPIXEL_DATA_FRONT
- LED1 pad 4: +5V -> /+5V_FRONT
- LED10 pad 2: Earth -> /GND_FRONT
- LED10 pad 4: +5V -> /+5V_FRONT
- LED11 pad 2: Earth -> /GND_FRONT
- LED11 pad 4: +5V -> /+5V_FRONT
- LED12 pad 2: Earth -> /GND_FRONT
- LED12 pad 4: +5V -> /+5V_FRONT
- LED2 pad 2: Earth -> /GND_FRONT
- LED2 pad 4: +5V -> /+5V_FRONT
- LED3 pad 2: Earth -> /GND_FRONT
- LED3 pad 4: +5V -> /+5V_FRONT
- LED4 pad 2: Earth -> /GND_FRONT
- LED4 pad 4: +5V -> /+5V_FRONT
- LED5 pad 2: Earth -> /GND_FRONT
- LED5 pad 4: +5V -> /+5V_FRONT
- LED6 pad 2: Earth -> /GND_FRONT
- LED6 pad 4: +5V -> /+5V_FRONT
- LED7 pad 2: Earth -> /GND_FRONT
- LED7 pad 4: +5V -> /+5V_FRONT
- LED8 pad 2: Earth -> /GND_FRONT
- LED8 pad 4: +5V -> /+5V_FRONT
- LED9 pad 2: Earth -> /GND_FRONT
- LED9 pad 4: +5V -> /+5V_FRONT
- P1 pad 1: IOVDD -> /GND_FRONT
- P1 pad 2: /KNOB_1 -> /KNOB_1_FRONT
- P1 pad 3: Earth -> /+3.3V_FRONT
- P2 pad 1: IOVDD -> /GND_FRONT
- P2 pad 2: /KNOB_2 -> /KNOB_2_FRONT
- P2 pad 3: Earth -> /+3.3V_FRONT
- R17 pad 1: Net-(J1-T) -> /CV_OUTPUT_1
- R18 pad 1: Net-(J2-T) -> /CV_OUTPUT_5
- R26 pad 1: Net-(J3-T) -> /CV_OUTPUT_2
- R27 pad 1: Net-(J4-T) -> /CV_OUTPUT_6
- R34 pad 1: Net-(J5-T) -> /CV_OUTPUT_3
- R35 pad 1: Net-(J6-T) -> /CV_OUTPUT_7
- R42 pad 1: Net-(J7-T) -> /CV_OUTPUT_4
- R43 pad 1: Net-(J8-T) -> /CV_OUTPUT_8
- R44 pad 1: Net-(J9-T) -> /CV_INPUT_1
- R47 pad 2: /INPUT_DETECT -> /INPUT_DETECT_FRONT
- R49 pad 2: /INPUT_DETECT -> /INPUT_DETECT_FRONT
- R51 pad 1: Net-(J10-T) -> /CV_INPUT_2
- R53 pad 2: /INPUT_DETECT -> /INPUT_DETECT_FRONT
- R55 pad 1: Net-(J11-T) -> /CV_INPUT_3
- R57 pad 2: /INPUT_DETECT -> /INPUT_DETECT_FRONT
- R59 pad 1: Net-(J12-T) -> /CV_INPUT_4
- R61 pad 1: Earth -> /GND_FRONT
- SW1 pad 1: /BUTTON_1 -> /BUTTON_1_FRONT
- SW1 pad 2: Earth -> /GND_FRONT
- SW2 pad 1: /BUTTON_2 -> /BUTTON_2_FRONT
- SW2 pad 2: Earth -> /GND_FRONT
Routing:
- net /+5V_FRONT: track 0.00 -> 189.3 mm, vias 0 -> 5
- net /GND_FRONT: track 0.00 -> 162.4 mm, vias 0 -> 16
- net /CV_OUTPUT_3_FRONT: track 0.00 -> 152.4 mm, vias 0 -> 2
- net /CV_OUTPUT_7_FRONT: track 0.00 -> 132.6 mm, vias 0 -> 1
- net /CV_OUTPUT_1_FRONT: track 0.00 -> 129.0 mm, vias 0 -> 1
- net /CV_OUTPUT_5_FRONT: track 0.00 -> 125.1 mm, vias 0 -> 1
- net /CV_OUTPUT_4_FRONT: track 0.00 -> 117.2 mm, vias 0 -> 2
- net /INPUT_DETECT_FRONT: track 0.00 -> 113.1 mm, vias 0 -> 3
- net /CV_INPUT_1_FRONT: track 0.00 -> 103.3 mm, vias 0 -> 1
- net /CV_OUTPUT_8_FRONT: track 0.00 -> 102.5 mm
- net /CV_OUTPUT_2_FRONT: track 0.00 -> 97.8 mm, vias 0 -> 2
- net /CV_INPUT_2_FRONT: track 0.00 -> 86.1 mm, vias 0 -> 2
- net /CV_INPUT_3_FRONT: track 0.00 -> 84.8 mm, vias 0 -> 1
- net /+3.3V_FRONT: track 0.00 -> 84.2 mm, vias 0 -> 2
- net /NEOPIXEL_DATA_FRONT: track 0.00 -> 82.8 mm, vias 0 -> 3
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- added copper zone on B.Cu, net /GND_FRONT
Other:
- board size 40.6 x 110 mm -> 87.6 x 110 mm

Commit message: kicad save
Parts:
- removed the U7 at (117.2, 31.1)
- added C25: 10u, Capacitor_SMD:C_0805_2012Metric, F.Cu at (71.6, 52.1)
- added C26: 10u, Capacitor_SMD:C_0805_2012Metric, F.Cu at (71.6, 59.7)
- added C30: 100n, Capacitor_SMD:C_0402_1005Metric, F.Cu at (47.5, 34.8)
- added D1: type="D" model="DIODE" lib="", Diode_SMD:D_SMA, F.Cu at (74.9, 51.9)
- added D2: type="D" model="DIODE" lib="", Diode_SMD:D_SMA, F.Cu at (74.9, 59.7)
- added J9: Conn_02x05_Odd_Even, Eurorack:Eurorack Power Header, B.Cu at (81.9, 49.5)
- JUMPER1, USB1: moved to B.Cu
- SW1: renamed from SW3; moved to B.Cu
- U6: renamed from U5; footprint Package_TO_SOT_SMD:TO-252-3_TabPin4 -> Package_SO:SOIC-8_5.23x5.23mm_P1.27mm
- moved D4 96.2 mm to (58.2, 12.4), turned to 90 degrees
- moved D3 94.0 mm to (59.4, 12.4), turned to -90 degrees
- moved DAC2 88.5 mm to (51.3, 49.0)
- moved DAC1 88.2 mm to (51.3, 42.9)
- moved C23 83.4 mm to (50.8, 19.1), turned to 90 degrees
- moved C11 81.1 mm to (47.6, 15.2)
- moved C19 80.2 mm to (47.6, 22.9)
- moved U1 78.5 mm to (59.6, 57.9)
- moved Y1 77.6 mm to (61.0, 29.0)
- moved U10 73.6 mm to (52.1, 32.8)
- moved C24 73.5 mm to (61.6, 22.2), turned to 180 degrees
- moved U5 72.3 mm to (50.2, 57.8), turned to 90 degrees
- moved C31 72.1 mm to (64.1, 19.1), turned to 180 degrees
- moved C10 70.0 mm to (48.8, 65.3)
- moved USB1 69.9 mm to (66.0, 67.3)
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- renumbered C9 to C10, C10 to C11, C11 to C12, C12 to C13, C13 to C14, C14 to C15, C15 to C16, C16 to C17, C17 to C18, C18 to C19, C19 to C20, C27 to C21, C28 to C22, C29 to C23, C30 to C24, C26 to C27, C20 to C28, C21 to C29, C22 to C31, C23 to C32, C25 to C33, C24 to C4, C4 to C5, C5 to C6, C6 to C7, C7 to C8, C8 to C9, D1 to D3, D2 to D4, J14 to J1, J3 to J10, J4 to J11, J5 to J12, J6 to J13, J7 to J14, J8 to J15, J13 to J16, J9 to J2, J11 to J3, J15 to J4, J1 to J5, J2 to J6, J12 to J7, J10 to J8, LED11 to LED10, LED10 to LED11, LED5 to LED2, LED2 to LED3, LED6 to LED4, LED3 to LED5, LED7 to LED6, LED4 to LED7, R9 to R10, R10 to R11, R11 to R12, R12 to R13, R13 to R14, R14 to R15, R47 to R16, R53 to R17, R15 to R18, R16 to R19, R17 to R20, R18 to R21, R48 to R22, R44 to R23, R54 to R24, R55 to R25, R19 to R26, R45 to R27, R56 to R28, R20 to R29, R46 to R3, R21 to R30, R22 to R31, R23 to R32, R24 to R33, R25 to R34, R57 to R35, R49 to R36, R26 to R37, R27 to R38, R58 to R39, R3 to R4, R59 to R40, R50 to R41, R51 to R42, R60 to R43, R52 to R44, R28 to R45, R29 to R46, R30 to R47, R31 to R48, R32 to R49, R4 to R5, R33 to R50, R34 to R51, R35 to R52, R36 to R53, R37 to R54, R38 to R55, R39 to R56, R40 to R57, R41 to R58, R61 to R59, R5 to R6, R42 to R60, R43 to R61, R6 to R7, R7 to R8, R8 to R9, SW1 to SW2, SW2 to SW3, U8 to U10, U11 to U3, U3 to U4, U4 to U5, U6 to U7, U7 to U8
Connections:
- net USB_DM renamed USB_DN
- U4 pad 12: unconnected-(U3-GPIO9-Pad12) -> /BUTTON_2
- U4 pad 13: unconnected-(U3-GPIO10-Pad13) -> /BUTTON_1
- U4 pad 14: unconnected-(U3-GPIO11-Pad14) -> /OLED_DIN
- U4 pad 16: unconnected-(U3-GPIO13-Pad16) -> /OLED_D/C
- U4 pad 17: unconnected-(U3-GPIO14-Pad17) -> /OLED_CLK
Routing:
- net /BUTTON_1: track 0.00 -> 78.2 mm, vias 0 -> 2
- net +5V: track 0.00 -> 76.4 mm, vias 0 -> 3
- net /KNOB_1: track 0.00 -> 66.4 mm, vias 0 -> 2
- net Net-(C28-Pad2): track 0.00 -> 65.6 mm, vias 0 -> 2
- net /OLED_D/C: track 0.00 -> 62.2 mm, vias 0 -> 2
- net /OLED_CLK: track 0.00 -> 59.6 mm, vias 0 -> 4
- net /CV_INPUT_3: track 0.00 -> 53.5 mm, vias 0 -> 4
- net Net-(C29-Pad2): track 0.00 -> 50.8 mm
- net Net-(C12-Pad2): track 0.00 -> 49.7 mm
- net /CV_INPUT_1: track 0.00 -> 45.6 mm, vias 0 -> 4
- net Net-(U9C-+): track 0.00 -> 44.9 mm, vias 0 -> 2
- net Net-(U9A-+): track 0.00 -> 43.8 mm, vias 0 -> 4
- net Net-(C11-Pad2): track 0.00 -> 43.7 mm, vias 0 -> 2
- net /NEOPIXEL_DATA: track 0.00 -> 43.6 mm, vias 0 -> 6
- net IOVDD: track 0.00 -> 41.8 mm, vias 0 -> 1
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Other:
- board size 87.6 x 110 mm -> 86.4 x 110 mm
- board text added: "BIPOLAR ±5V"
- board text added: "MCP3428 ADC"
- board text added: "MCP6004"
- board text added: "TL074 1-4"
- board text added: "TL074 5-8"
- board text added: "UNIPOLAR 0-10V"

Commit message: kicad save
Parts:
- removed J1: Conn_02x12_Counter_Clockwise, Connector_PinSocket_2.54mm:PinSocket_2x12_P2.54mm_Vertical
- removed R16, R17, R35, R36: 10K, Resistor_SMD:R_0402_1005Metric
- removed R6, R7: 5K1, Resistor_SMD:R_0402_1005Metric
- removed SW1: BOOT, Button_Switch_THT:SW_PUSH_6mm_H4.3mm
- removed USB1: USB_C_Receptacle_USB2.0, Connector_USB:USB_C_Receptacle_Amphenol_12401548E4-2A
- added C34: 10u, Capacitor_SMD:C_0805_2012Metric, F.Cu at (72.1, 46.6)
- added D5: type="D" model="DIODE" lib="", Diode_SMD:D_SMA, F.Cu at (75.4, 46.7)
- added J17: Conn_02x08_Odd_Even, Eurorack:Eurorack Power Header 16 Pin, B.Cu at (81.8, 55.6)
- added J18: Conn_01x16_Pin, Connector_PinHeader_2.54mm:PinHeader_1x16_P2.54mm_Vertical, B.Cu at (39.4, 1.27)
- added J19: Conn_01x16_Pin, Connector_PinSocket_2.54mm:PinSocket_1x16_P2.54mm_Vertical, F.Cu at (85.1, 1.27)
- added J20: Conn_01x06_Pin, Connector_PinHeader_2.54mm:PinHeader_1x06_P2.54mm_Horizontal, B.Cu at (71.1, 74.9)
- added TP1: TestPoint, TestPoint:TestPoint_Pad_1.0x1.0mm, B.Cu at (51.6, 83.8)
- added TP2: TestPoint, TestPoint:TestPoint_Pad_1.0x1.0mm, B.Cu at (49.3, 83.8)
- added TP3: TestPoint, TestPoint:TestPoint_Pad_1.0x1.0mm, B.Cu at (47.0, 83.8)
- added TP4: TestPoint, TestPoint:TestPoint_Pad_1.0x1.0mm, B.Cu at (56.1, 83.8)
- added TP5: TestPoint, TestPoint:TestPoint_Pad_1.0x1.0mm, B.Cu at (53.8, 83.8)
- added TP6: TestPoint, TestPoint:TestPoint_Pad_1.0x1.0mm, F.Cu at (58.9, 37.3)
- added TP7: TestPoint, TestPoint:TestPoint_Pad_1.0x1.0mm, F.Cu at (61.1, 37.3)
- added TP8: TestPoint, TestPoint:TestPoint_Pad_1.0x1.0mm, F.Cu at (78.0, 38.6)
- J4: value Conn_02x12_Counter_Clockwise -> Conn_01x16_Pin; footprint Connector_PinHeader_2.54mm:PinHeader_2x12_P2.54mm_Vertical -> Connector_PinSocket_2.54mm:PinSocket_1x16_P2.54mm_Vertical; moved to F.Cu
- J9: value Conn_02x05_Odd_Even -> Conn_01x16_Pin; footprint Eurorack:Eurorack Power Header -> Connector_PinHeader_2.54mm:PinHeader_1x16_P2.54mm_Vertical
- moved J9 94.0 mm to (1.27, 1.27), turned to 180 degrees
- moved JUMPER1 60.7 mm to (61.0, 83.8), turned to -90 degrees
- moved R59 58.4 mm to (82.4, 27.1), turned to -90 degrees
- moved C33 54.5 mm to (81.0, 27.1), turned to 90 degrees
- moved DAC2 40.9 mm to (61.5, 9.40)
- moved DAC1 39.7 mm to (61.5, 4.57)
- moved D3 39.4 mm to (64.0, 51.6)
- moved D4 39.3 mm to (62.2, 51.6)
- moved R24 37.3 mm to (51.8, 25.4), turned to 0 degrees
- moved R25 32.6 mm to (51.8, 24.1), turned to 0 degrees
- moved R28 30.8 mm to (51.8, 22.9), turned to 180 degrees
- moved C11 29.9 mm to (74.7, 2.54), turned to 180 degrees
- moved R12 29.8 mm to (76.5, 3.05), turned to -90 degrees
- moved C27 29.2 mm to (49.5, 18.0), turned to -90 degrees
- moved R39 27.5 mm to (54.4, 25.4), turned to 180 degrees
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Connections:
- C11 pad 1: Net-(U7A-+) -> Net-(U7D-+)
- C12 pad 1: Net-(U8A-+) -> Net-(U8D-+)
- C19 pad 1: Net-(U7B-+) -> Net-(U7A-+)
- C20 pad 1: Net-(U8B-+) -> Net-(U8A-+)
- C28 pad 1: Net-(U7C-+) -> Net-(U7B-+)
- C29 pad 1: Net-(U8C-+) -> Net-(U8B-+)
- C31 pad 1: Net-(U7D-+) -> Net-(U7C-+)
- C32 pad 1: Net-(U8D-+) -> Net-(U8C-+)
- C33 pad 2: /GND_FRONT -> Earth
- J16 pad 20: /D2 -> unconnected-(J16-Pin_20-Pad20)
- J16 pad 26: /IREF -> /IREF_FRONT
- J16 pad 27: /VCOMH -> /VCOMH_FRONT
- J2 pad 2: Net-(J2-TN) -> /INPUT_DETECT_FRONT
- J3 pad 2: Net-(J3-TN) -> /INPUT_DETECT_FRONT
- J4 pad 1: /+5V_FRONT -> Earth
- J4 pad 10: /CV_OUTPUT_3_FRONT -> /KNOB_2
- J4 pad 11: /CV_OUTPUT_4_FRONT -> /KNOB_1
- J4 pad 12: /CV_OUTPUT_5_FRONT -> /BUTTON_2
- J4 pad 13: /CV_OUTPUT_6_FRONT -> /BUTTON_1
- J4 pad 14: /CV_OUTPUT_7_FRONT -> Earth
- J4 pad 15: /CV_OUTPUT_8_FRONT -> IOVDD
- J4 pad 16: /BUTTON_1_FRONT -> +5V
- J4 pad 2: /+3.3V_FRONT -> Earth
- J4 pad 3: /GND_FRONT -> Earth
- J4 pad 4: /CV_INPUT_1_FRONT -> Earth
- J4 pad 5: /CV_INPUT_2_FRONT -> Earth
- J4 pad 6: /CV_INPUT_3_FRONT -> /CV_INPUT_1
- J4 pad 7: /CV_INPUT_4_FRONT -> /CV_INPUT_2
- J4 pad 8: /CV_OUTPUT_1_FRONT -> /CV_INPUT_3
- J4 pad 9: /CV_OUTPUT_2_FRONT -> /CV_INPUT_4
- J7 pad 2: Net-(J7-TN) -> /INPUT_DETECT_FRONT
- J8 pad 2: Net-(J8-TN) -> /INPUT_DETECT_FRONT
- J9 pad 1: Net-(D2-K) -> /GND_FRONT
- J9 pad 10: Net-(D1-A) -> /KNOB_2_FRONT
- J9 pad 2: Net-(D2-K) -> /GND_FRONT
- J9 pad 3: Earth -> /GND_FRONT
- J9 pad 4: Earth -> /GND_FRONT
- J9 pad 5: Earth -> /GND_FRONT
- J9 pad 6: Earth -> /CV_INPUT_1_FRONT
- J9 pad 7: Earth -> /CV_INPUT_2_FRONT
- J9 pad 8: Earth -> /CV_INPUT_3_FRONT
- J9 pad 9: Net-(D1-A) -> /CV_INPUT_4_FRONT
- R11 pad 2: Net-(R11-Pad2) -> /BOOTSEL
- R12 pad 1: Net-(U7A-+) -> Net-(U7D-+)
- R13 pad 1: Net-(U7A-+) -> Net-(U7D-+)
- R14 pad 1: Net-(U8A-+) -> Net-(U8D-+)
- R15 pad 1: Net-(U8A-+) -> Net-(U8D-+)
- R18 pad 2: Net-(U7A-+) -> Net-(U7D-+)
- R19 pad 2: Net-(U8A-+) -> Net-(U8D-+)
- R27 pad 2: /CV_INPUT_1 -> /ADC_INPUT_1
- R28 pad 2: /CV_INPUT_3 -> /ADC_INPUT_3
- R29 pad 1: Net-(U7B-+) -> Net-(U7A-+)
- R30 pad 1: Net-(U7B-+) -> Net-(U7A-+)
- R31 pad 1: Net-(U8B-+) -> Net-(U8A-+)
- R32 pad 1: Net-(U8B-+) -> Net-(U8A-+)
- R33 pad 2: Net-(U7B-+) -> Net-(U7A-+)
- R34 pad 2: Net-(U8B-+) -> Net-(U8A-+)
- R43 pad 2: /CV_INPUT_4 -> /ADC_INPUT_4
- R44 pad 2: /CV_INPUT_2 -> /ADC_INPUT_2
- R45 pad 1: Net-(U7C-+) -> Net-(U7B-+)
- R46 pad 1: Net-(U7C-+) -> Net-(U7B-+)
- R47 pad 1: Net-(U8C-+) -> Net-(U8B-+)
- R48 pad 1: Net-(U8C-+) -> Net-(U8B-+)
- R49 pad 2: Net-(U7C-+) -> Net-(U7B-+)
- R50 pad 2: Net-(U8C-+) -> Net-(U8B-+)
- R53 pad 1: Net-(U7D-+) -> Net-(U7C-+)
- R54 pad 1: Net-(U7D-+) -> Net-(U7C-+)
- R55 pad 1: Net-(U8D-+) -> Net-(U8C-+)
- R56 pad 1: Net-(U8D-+) -> Net-(U8C-+)
- R57 pad 2: Net-(U7D-+) -> Net-(U7C-+)
- R58 pad 2: Net-(U8D-+) -> Net-(U8C-+)
- R59 pad 1: /GND_FRONT -> Earth
- U10 pad 1: /CV_INPUT_1 -> /ADC_INPUT_1
- U10 pad 11: /CV_INPUT_3 -> /ADC_INPUT_3
- U10 pad 13: /CV_INPUT_4 -> /ADC_INPUT_4
- U10 pad 3: /CV_INPUT_2 -> /ADC_INPUT_2
- U4 pad 26: RUN -> /RUN
- U7 pad 1: Net-(C11-Pad2) -> Net-(C19-Pad2)
- U7 pad 14: Net-(C31-Pad2) -> Net-(C11-Pad2)
- U7 pad 7: Net-(C19-Pad2) -> Net-(C28-Pad2)
- U7 pad 8: Net-(C28-Pad2) -> Net-(C31-Pad2)
- U8 pad 1: Net-(C12-Pad2) -> Net-(C20-Pad2)
- U8 pad 14: Net-(C32-Pad2) -> Net-(C12-Pad2)
- U8 pad 7: Net-(C20-Pad2) -> Net-(C29-Pad2)
- U8 pad 8: Net-(C29-Pad2) -> Net-(C32-Pad2)
- U9 pad 1: /CV_INPUT_1 -> /ADC_INPUT_1
- U9 pad 14: /CV_INPUT_4 -> /ADC_INPUT_4
- U9 pad 7: /CV_INPUT_2 -> /ADC_INPUT_2
- U9 pad 8: /CV_INPUT_3 -> /ADC_INPUT_3
Routing:
- net Earth: track 0.00 -> 185.7 mm, vias 0 -> 46
- net -12V: track 9.27 -> 165.7 mm, vias 0 -> 12
- net IOVDD: track 41.8 -> 194.5 mm, vias 1 -> 16
- net /DAC_OFFSET: track 0.00 -> 122.2 mm, vias 0 -> 11
- net +12V: track 8.98 -> 130.7 mm, vias 0 -> 10
- net /GND_FRONT: track 162.4 -> 78.8 mm
- net /RUN: track 0.00 -> 70.4 mm, vias 0 -> 2
- net /I2C1_SCL: track 0.00 -> 67.0 mm, vias 0 -> 4
- net /I2C1_SDA: track 0.00 -> 66.3 mm, vias 0 -> 4
- net /I2C0_SDA: track 9.04 -> 72.7 mm, vias 2 -> 8
- net /-4.096VREF: track 8.43 -> 68.0 mm, vias 0 -> 1
- net Net-(C28-Pad2): track 65.6 -> 7.70 mm, vias 2 -> 0
- net /I2C0_SCL: track 10.8 -> 67.4 mm, vias 2 -> 8
- net /IREF_FRONT: track 0.00 -> 55.0 mm, vias 0 -> 2
- net /-2.048VREF: track 7.55 -> 62.1 mm, vias 0 -> 1
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- added copper zone on B.Cu, net Earth
Other:
- board size 86.4 x 110 mm -> 86.4 x 110.1 mm
- board text added: "+12V"
- board text added: "+3.3V"
- board text added: "+3.3V REG"
- board text added: "+5V"
- board text added: "-10V"
- board text added: "-12V"
- board text added: "-2.048V"
- board text added: "-4.096V"
- board text added: "3.3V"
- board text added: "GND"
- board text added: "I2C FROM RP2040"
- board text added: "I2C TO RP2040"
- board text added: "INPUT ADC"
- board text added: "INPUT CONDITIONING"
- board text added: "OUTPUT CONDITIONING"
- board text added: "OUTPUT DACS"
- board text added: "VREF"
- board text added: "VREFS"
- board text added: "±10V from jacks"
- board text added: "±5V OR 0-10V to jacks"
- board text removed: "MCP3428 ADC"
- board text removed: "MCP6004"
- board text removed: "TL074 1-4"
- board text removed: "TL074 5-8"
