File: hardware/EuroPi-X/kicad/EuroPi-X.kicad_sch (KiCad schematic)
At the start: 88 parts, among them J1 USB_C_Receptacle_USB2.0, J10 Thonkiconn_Mono_Jack, J11 Thonkiconn_Mono_Jack, J12 Thonkiconn_Mono_Jack, J13 Thonkiconn_Mono_Jack, J14 Thonkiconn_Mono_Jack, J3 Thonkiconn_Mono_Jack, J7 UNI/BIPOLAR, J8 Thonkiconn_Mono_Jack, J9 Thonkiconn_Mono_Jack, SW2 BOOT, U1 RP2040, U4 TL074, U5 TL074, U6 LM4030-4.096, U7 LM4040DBZ-2.0, U8 TL074, Y1 Crystal_GND2

Commit message: kicad save
Parts:
- added C24: 1u, Capacitor_SMD:C_0402_1005Metric, symbol Device:C
- added C25: 100n, Capacitor_SMD:C_0402_1005Metric, symbol Device:C
- added D1, D2: D, Diode_SMD:D_0402_1005Metric, symbol Device:D
- added J10, J11, J12, J9: Thonkiconn_Mono_Jack, Eurorack:Thonkiconn Mono Jack, symbol Eurorack:Thonkiconn_Mono_Jack
- added J13: Conn_01x30_Pin, Connector_FFC-FPC:Hirose_FH41-30S-0.5SH_1x30_1MP_1SH_P0.5mm_Horizontal, symbol Connector:Conn_01x30_Pin
- added LED1, LED10, LED11, LED12, LED2, LED3, LED4, LED5, LED6, LED7, LED8, LED9: SK6805, LED_SMD:LED_SK6805_PLCC4_2.4x2.7mm_P1.3mm, symbol LED:SK6805
- added P1, P2: Potentiometer_9mm_Vertical_Linear, Eurorack:Potentiometer 9mm Vertical Linear Centred, symbol Eurorack:Potentiometer_9mm_Vertical_Linear
- added R44, R48, R50, R51, R54, R55, R58, R59: 100K, Resistor_SMD:R_0402_1005Metric, symbol Device:R
- added R45, R52, R56, R60: 15K, Resistor_SMD:R_0402_1005Metric, symbol Device:R
- added R46: 2K2, Resistor_SMD:R_0402_1005Metric, symbol Device:R
- added R47, R49, R53, R57: 10K, Resistor_SMD:R_0402_1005Metric, symbol Device:R
- added R61: ~, Resistor_SMD:R_0402_1005Metric, symbol Device:R
- added SW1, SW2: BOOT, Eurorack:Switch Tactile Momentary C&K, symbol Switch:SW_Push
- added U11: LM4040DBZ-10, Package_TO_SOT_SMD:SOT-23, symbol Reference_Voltage:LM4040DBZ-10
- added U8: MCP3428, Package_SO:SOIC-14_3.9x8.7mm_P1.27mm, symbol Analog_ADC:MCP3428
- added U9: MCP6004, Package_SO:TSSOP-14_4.4x5mm_P0.65mm, symbol Amplifier_Operational:MCP6004
- C10: renamed from C14; footprint (none) -> Capacitor_SMD:C_0402_1005Metric
- C11: renamed from C20; footprint (none) -> Capacitor_SMD:C_0402_1005Metric
- C18: renamed from C17; footprint (none) -> Capacitor_SMD:C_0402_1005Metric
- C19: renamed from C21; footprint (none) -> Capacitor_SMD:C_0402_1005Metric
- C20: renamed from C18; footprint (none) -> Capacitor_SMD:C_0402_1005Metric
- C21: renamed from C22; footprint (none) -> Capacitor_SMD:C_0402_1005Metric
- C22: renamed from C19; footprint (none) -> Capacitor_SMD:C_0402_1005Metric
- C23: footprint (none) -> Capacitor_SMD:C_0402_1005Metric
- JUMPER1: renamed from J7; footprint (none) -> Connector_PinHeader_2.54mm:PinHeader_1x03_P2.54mm_Vertical
- R1: renamed from R15; footprint (none) -> Resistor_SMD:R_0402_1005Metric
- R11: renamed from R12; footprint (none) -> Resistor_SMD:R_0402_1005Metric
- R12: renamed from R11; footprint (none) -> Resistor_SMD:R_0402_1005Metric
- R13: renamed from R29; footprint (none) -> Resistor_SMD:R_0402_1005Metric
- R14: renamed from R30; footprint (none) -> Resistor_SMD:R_0402_1005Metric
- R15: renamed from R13; footprint (none) -> Resistor_SMD:R_0402_1005Metric
- R16: renamed from R31; footprint (none) -> Resistor_SMD:R_0402_1005Metric
- R17: renamed from R14; footprint (none) -> Resistor_SMD:R_0402_1005Metric
- R18: renamed from R32; footprint (none) -> Resistor_SMD:R_0402_1005Metric
- R2: renamed from R16; footprint (none) -> Resistor_SMD:R_0402_1005Metric
- R20: renamed from R17; footprint (none) -> Resistor_SMD:R_0402_1005Metric
- R21: renamed from R18; footprint (none) -> Resistor_SMD:R_0402_1005Metric
- R22: renamed from R33; footprint (none) -> Resistor_SMD:R_0402_1005Metric
- R23: renamed from R34; footprint (none) -> Resistor_SMD:R_0402_1005Metric
- R24: renamed from R19; footprint (none) -> Resistor_SMD:R_0402_1005Metric
- R25: renamed from R35; footprint (none) -> Resistor_SMD:R_0402_1005Metric
- R26: renamed from R20; footprint (none) -> Resistor_SMD:R_0402_1005Metric
- R27: renamed from R36; footprint (none) -> Resistor_SMD:R_0402_1005Metric
- R28: renamed from R21; footprint (none) -> Resistor_SMD:R_0402_1005Metric
- R29: renamed from R22; footprint (none) -> Resistor_SMD:R_0402_1005Metric
- R30: renamed from R37; footprint (none) -> Resistor_SMD:R_0402_1005Metric
- R31: renamed from R38; footprint (none) -> Resistor_SMD:R_0402_1005Metric
- R32: renamed from R23; footprint (none) -> Resistor_SMD:R_0402_1005Metric
- R33: renamed from R39; footprint (none) -> Resistor_SMD:R_0402_1005Metric
- R34: renamed from R24; footprint (none) -> Resistor_SMD:R_0402_1005Metric
- R35: renamed from R40; footprint (none) -> Resistor_SMD:R_0402_1005Metric
- R36: renamed from R25; footprint (none) -> Resistor_SMD:R_0402_1005Metric
- R37: renamed from R26; footprint (none) -> Resistor_SMD:R_0402_1005Metric
- R38: renamed from R41; footprint (none) -> Resistor_SMD:R_0402_1005Metric
- R39: renamed from R42; footprint (none) -> Resistor_SMD:R_0402_1005Metric
- R40: renamed from R27; footprint (none) -> Resistor_SMD:R_0402_1005Metric
- R41: renamed from R43; footprint (none) -> Resistor_SMD:R_0402_1005Metric
- R42: renamed from R28; footprint (none) -> Resistor_SMD:R_0402_1005Metric
- R43: renamed from R44; footprint (none) -> Resistor_SMD:R_0402_1005Metric
- R7: renamed from R10; footprint (none) -> Resistor_SMD:R_0402_1005Metric
- R8: renamed from R9; footprint (none) -> Resistor_SMD:R_0402_1005Metric
- SW3: renamed from SW2; footprint Button_Switch_SMD:SW_SP3T_PCM13 -> Button_Switch_THT:SW_PUSH_6mm_H4.3mm
- U6: renamed from U4; footprint (none) -> Package_SO:SOIC-16_3.9x9.9mm_P1.27mm
- U7: renamed from U5; footprint (none) -> Package_SO:SOIC-16_3.9x9.9mm_P1.27mm
- U7: renamed from U8; footprint (none) -> Package_SO:SOIC-16_3.9x9.9mm_P1.27mm
- renumbered C6 to C12, C7 to C13, C8 to C14, C9 to C15, C10 to C16, C11 to C17, C15 to C2, C16 to C3, C2 to C4, C3 to C5, C4 to C6, C12 to C7, C13 to C8, C5 to C9, J3 to J1, J11 to J2, J8 to J3, J12 to J4, J9 to J5, J13 to J6, J10 to J7, J14 to J8, R8 to R10, R7 to R19, R1 to R3, R2 to R4, R3 to R5, R4 to R6, R6 to R9, U6 to U1, U7 to U2, U1 to U3, U2 to U4, U3 to U5, J1 to USB1
Connections:
- net +3V3 is gone; now on net +3.3V: C13.1, C15.1, C16.1, C17.1, C9.1, R19.1, R9.1, U3.1 (IOVDD), U3.10 (IOVDD), U3.2 (GPIO0), U3.22 (IOVDD), U3.33 (IOVDD), U3.42 (IOVDD), U3.48 (USB_VDD), U3.49 (IOVDD), U4.1 (OUT), U5.8 (VCC)
- net +3.3V: now also D1.1 (K), J13.10 (Pin_10), J13.14 (Pin_14), J13.28 (Pin_28), J13.6 (Pin_6), J13.9 (Pin_9), P1.1, P2.1, U8.6 (VDD), U9.4 (V+)
- net +5V: now also LED1.4 (VDD), LED10.4 (VDD), LED11.4 (VDD), LED12.4 (VDD), LED2.4 (VDD), LED3.4 (VDD), LED4.4 (VDD), LED5.4 (VDD), LED6.4 (VDD), LED7.4 (VDD), LED8.4 (VDD), LED9.4 (VDD)
- net -12V: now also R46.2
- net Earth: now also C24.2, C25.2, D2.2 (A), J10.1 (E), J11.1 (E), J12.1 (E), J13.11 (Pin_11), J13.12 (Pin_12), J13.13 (Pin_13), J13.16 (Pin_16), J13.17 (Pin_17), J13.21 (Pin_21), J13.22 (Pin_22), J13.23 (Pin_23), J13.24 (Pin_24), J13.25 (Pin_25), J13.29 (Pin_29), J13.8 (Pin_8), J9.1 (E), LED1.2 (VSS), LED10.2 (VSS), LED11.2 (VSS), LED12.2 (VSS), LED2.2 (VSS), LED3.2 (VSS), LED4.2 (VSS), LED5.2 (VSS), LED6.2 (VSS), LED7.2 (VSS), LED8.2 (VSS), LED9.2 (VSS), P1.3, P2.3, R61.1, SW1.2, SW2.2, U11.1 (K), U8.10 (Adr1), U8.12 (CH3-), U8.14 (CH4-), U8.2 (CH1-), U8.4 (CH2-), U8.5 (VSS), U8.9 (Adr0), U9.11 (V-), U9.13 (-), U9.2 (-), U9.6 (-), U9.9 (-)
- net NEOPIXEL_DATA: now reaches U3.11 (GPIO8)
- net NEOPIXEL_DATA: now also LED1.3 (DIN)
- net KNOB_1: now reaches U3.38 (GPIO26_ADC0)
- net KNOB_1: now also P1.2
- net KNOB_2: now reaches U3.39 (GPIO27_ADC1)
- net KNOB_2: now also P2.2
- net INPUT_DETECT: now reaches U3.5 (GPIO3)
- net INPUT_DETECT: now also D1.2 (A), D2.1 (K), R47.2, R49.2, R53.2, R57.2
- net I2C0_SDA: now reaches U3.6 (GPIO4)
- net I2C0_SDA: now also DAC1.3 (SDA), U8.7 (SDA)
- net I2C0_SCL: now reaches U3.7 (GPIO5)
- net I2C0_SCL: now also DAC1.2 (SCL), U8.8 (SCL)
- net I2C1_SDA: now reaches U3.8 (GPIO6)
- net I2C1_SDA: now also DAC2.3 (SDA)
- net I2C1_SCL: now reaches U3.9 (GPIO7)
- net I2C1_SCL: now also DAC2.2 (SCL)
- net DAC_1_SCL: no longer names the net of U3.28 (GPIO17)
- net DAC_1_SCL: no longer DAC1.2 (SCL)
- net DAC_1_SDA: no longer names the net of U3.27 (GPIO16)
- net DAC_1_SDA: no longer DAC1.3 (SDA)
- net DAC_2_SCL: no longer names the net of U3.30 (GPIO19)
- net DAC_2_SCL: no longer DAC2.2 (SCL)
- net DAC_2_SDA: no longer names the net of U3.29 (GPIO18)
- net DAC_2_SDA: no longer DAC2.3 (SDA)
- new net: J11.3 (T), R55.1
- new net: R54.2, R55.2, R56.1, U9.10 (+)
- new net: LED10.3 (DIN), LED9.1 (DOUT)
- new net: LED8.1 (DOUT), LED9.3 (DIN)
- new net: R44.2, R45.1, R48.2, U9.3 (+)
- new net: J11.2 (TN), R53.1
- new net: J12.2 (TN), R57.1
- new net: J12.3 (T), R59.1
- new net: R58.2, R59.2, R60.1, U9.12 (+)
- new net: LED1.1 (DOUT), LED2.3 (DIN)
- new net: LED10.1 (DOUT), LED11.3 (DIN)
- new net: R50.2, R51.2, R52.1, U9.5 (+)
- new net: LED3.1 (DOUT), LED4.3 (DIN)
- new net: LED2.1 (DOUT), LED3.3 (DIN)
- new net: J10.2 (TN), R49.1
- new net: LED4.1 (DOUT), LED5.3 (DIN)
- new net: LED11.1 (DOUT), LED12.3 (DIN)
- new net: LED7.1 (DOUT), LED8.3 (DIN)
- new net: LED6.1 (DOUT), LED7.3 (DIN)
- new net: LED5.1 (DOUT), LED6.3 (DIN)
- new net: J9.2 (TN), R47.1
- new net: J9.3 (T), R44.1
- new net: J10.3 (T), R51.1
- new net -10VREF: C24.1, R46.1, R48.1, R50.1, R54.1, R58.1, U11.2 (A)
- new net BUTTON_1: SW1.1
- new net BUTTON_2: SW2.1
- new net CV_INPUT_1: R45.2, U8.1 (CH1+), U9.1
- new net CV_INPUT_2: R52.2, U8.3 (CH2+), U9.7
- new net CV_INPUT_3: R56.2, U8.11 (CH3+), U9.8
- new net CV_INPUT_4: R60.2, U8.13 (CH4+), U9.14
- new net D0: J13.18 (Pin_18)
- new net D1: J13.19 (Pin_19)
- new net D2: J13.20 (Pin_20)
- new net D/C#: J13.15 (Pin_15)
- new net IREF: J13.26 (Pin_26), R61.2
- new net VCOMH: C25.1, J13.27 (Pin_27)
- no-connect marks 10 -> 17
Other:
- note added: "-10V REFERENCE"
- note added: "BUTTONS"
- note added: "INPUT ADCS"
- note added: "INPUT DETECTION"
- note added: "INPUTS"
- note added: "KNOBS"
- note added: "OLED"

Commit message: kicad save and pdf schematic
Parts:
- added C26, C27, C28, C29, C30: 100n, Capacitor_SMD:C_0402_1005Metric, symbol Device:C
- added J14: Conn_02x12_Counter_Clockwise, Connector_PinSocket_2.54mm:PinSocket_2x12_P2.54mm_Vertical, symbol Connector_Generic:Conn_02x12_Counter_Clockwise
- added J15: Conn_02x12_Counter_Clockwise, Connector_PinHeader_2.54mm:PinHeader_2x12_P2.54mm_Vertical, symbol Connector_Generic:Conn_02x12_Counter_Clockwise
Connections:
- net +12V: now also C27.1, C29.1
- net +3.3V: now also C26.1, J14.3 (Pin_3); no longer J13.10 (Pin_10), J13.14 (Pin_14), J13.28 (Pin_28), J13.6 (Pin_6), J13.9 (Pin_9), P1.1, P2.1
- net +5V: now also J14.2 (Pin_2); no longer LED1.4 (VDD), LED10.4 (VDD), LED11.4 (VDD), LED12.4 (VDD), LED2.4 (VDD), LED3.4 (VDD), LED4.4 (VDD), LED5.4 (VDD), LED6.4 (VDD), LED7.4 (VDD), LED8.4 (VDD), LED9.4 (VDD)
- net -12V: now also C28.2, C30.2
- net BUTTON_1: now also J14.16 (Pin_16); no longer SW1.1
- net BUTTON_2: now also J14.17 (Pin_17); no longer SW2.1
- net CV_INPUT_1: now also R44.1, J14.4 (Pin_4)
- net CV_INPUT_2: now also R51.1, J14.5 (Pin_5)
- net CV_INPUT_3: now also R55.1, J14.6 (Pin_6)
- net CV_INPUT_4: now also R59.1, J14.7 (Pin_7)
- net Earth: now also C26.2, C27.2, C28.1, C29.2, C30.1, J14.1 (Pin_1); no longer C25.2, J1.1 (E), J10.1 (E), J11.1 (E), J12.1 (E), J13.11 (Pin_11), J13.12 (Pin_12), J13.13 (Pin_13), J13.16 (Pin_16), J13.17 (Pin_17), J13.21 (Pin_21), J13.22 (Pin_22), J13.23 (Pin_23), J13.24 (Pin_24), J13.25 (Pin_25), J13.29 (Pin_29), J13.8 (Pin_8), J2.1 (E), J3.1 (E), J4.1 (E), J5.1 (E), J6.1 (E), J7.1 (E), J8.1 (E), J9.1 (E), LED1.2 (VSS), LED10.2 (VSS), LED11.2 (VSS), LED12.2 (VSS), LED2.2 (VSS), LED3.2 (VSS), LED4.2 (VSS), LED5.2 (VSS), LED6.2 (VSS), LED7.2 (VSS), LED8.2 (VSS), LED9.2 (VSS), P1.3, P2.3, R61.1, SW1.2, SW2.2
- net INPUT_DETECT: now also J14.24 (Pin_24); no longer R47.2, R49.2, R53.2, R57.2
- net KNOB_1: now also J14.18 (Pin_18); no longer P1.2
- net KNOB_2: now also J14.19 (Pin_19); no longer P2.2
- net NEOPIXEL_DATA: now also J14.23 (Pin_23); no longer LED1.3 (DIN)
- net CV_INPUT_3_FRONT: now reaches J11.3 (T)
- net CV_INPUT_3_FRONT: now also J15.6 (Pin_6); no longer R55.1
- net CV_INPUT_4_FRONT: now reaches J12.3 (T)
- net CV_INPUT_4_FRONT: now also J15.7 (Pin_7); no longer R59.1
- net CV_OUTPUT_7: now reaches R35.1
- net CV_OUTPUT_7: now also J14.14 (Pin_14); no longer J6.3 (T)
- net CV_OUTPUT_8: now reaches R43.1
- net CV_OUTPUT_8: now also J14.15 (Pin_15); no longer J8.3 (T)
- net CV_OUTPUT_3: now reaches R34.1
- net CV_OUTPUT_3: now also J14.10 (Pin_10); no longer J5.3 (T)
- net CV_OUTPUT_4: now reaches R42.1
- net CV_OUTPUT_4: now also J14.11 (Pin_11); no longer J7.3 (T)
- net CV_OUTPUT_1: now reaches R17.1
- net CV_OUTPUT_1: now also J14.8 (Pin_8); no longer J1.3 (T)
- net CV_OUTPUT_5: now reaches R18.1
- net CV_OUTPUT_5: now also J14.12 (Pin_12); no longer J2.3 (T)
- net CV_OUTPUT_2: now reaches R26.1
- net CV_OUTPUT_2: now also J14.9 (Pin_9); no longer J3.3 (T)
- net CV_OUTPUT_6: now reaches R27.1
- net CV_OUTPUT_6: now also J14.13 (Pin_13); no longer J4.3 (T)
- net CV_INPUT_1_FRONT: now reaches J9.3 (T)
- net CV_INPUT_1_FRONT: now also J15.4 (Pin_4); no longer R44.1
- net CV_INPUT_2_FRONT: now reaches J10.3 (T)
- net CV_INPUT_2_FRONT: now also J15.5 (Pin_5); no longer R51.1
- net D0 renamed OLED_CLK_FRONT
- net OLED_CLK_FRONT: now also J15.22 (Pin_22)
- net D1 renamed OLED_DIN_FRONT
- net OLED_DIN_FRONT: now also J15.21 (Pin_21)
- net D/C# renamed OLED_D/C_FRONT
- net OLED_D/C_FRONT: now also J15.20 (Pin_20)
- new net +3.3V_FRONT: J13.10 (Pin_10), J13.14 (Pin_14), J13.28 (Pin_28), J13.6 (Pin_6), J13.9 (Pin_9), J15.2 (Pin_2), P1.3, P2.3
- new net +5V_FRONT: J15.1 (Pin_1), LED1.4 (VDD), LED10.4 (VDD), LED11.4 (VDD), LED12.4 (VDD), LED2.4 (VDD), LED3.4 (VDD), LED4.4 (VDD), LED5.4 (VDD), LED6.4 (VDD), LED7.4 (VDD), LED8.4 (VDD), LED9.4 (VDD)
- new net BUTTON_1_FRONT: J15.16 (Pin_16), SW1.1
- new net BUTTON_2_FRONT: J15.17 (Pin_17), SW2.1
- new net CV_OUTPUT_1_FRONT: J1.3 (T), J15.8 (Pin_8)
- new net CV_OUTPUT_2_FRONT: J15.9 (Pin_9), J3.3 (T)
- new net CV_OUTPUT_3_FRONT: J15.10 (Pin_10), J5.3 (T)
- new net CV_OUTPUT_4_FRONT: J15.11 (Pin_11), J7.3 (T)
- new net CV_OUTPUT_5_FRONT: J15.12 (Pin_12), J2.3 (T)
- new net CV_OUTPUT_6_FRONT: J15.13 (Pin_13), J4.3 (T)
- new net CV_OUTPUT_7_FRONT: J15.14 (Pin_14), J6.3 (T)
- new net CV_OUTPUT_8_FRONT: J15.15 (Pin_15), J8.3 (T)
- new net GND_FRONT: C25.2, J1.1 (E), J10.1 (E), J11.1 (E), J12.1 (E), J13.11 (Pin_11), J13.12 (Pin_12), J13.13 (Pin_13), J13.16 (Pin_16), J13.17 (Pin_17), J13.21 (Pin_21), J13.22 (Pin_22), J13.23 (Pin_23), J13.24 (Pin_24), J13.25 (Pin_25), J13.29 (Pin_29), J13.8 (Pin_8), J15.3 (Pin_3), J2.1 (E), J3.1 (E), J4.1 (E), J5.1 (E), J6.1 (E), J7.1 (E), J8.1 (E), J9.1 (E), LED1.2 (VSS), LED10.2 (VSS), LED11.2 (VSS), LED12.2 (VSS), LED2.2 (VSS), LED3.2 (VSS), LED4.2 (VSS), LED5.2 (VSS), LED6.2 (VSS), LED7.2 (VSS), LED8.2 (VSS), LED9.2 (VSS), P1.1, P2.1, R61.1, SW1.2, SW2.2
- new net INPUT_DETECT_FRONT: J15.24 (Pin_24), R47.2, R49.2, R53.2, R57.2
- new net KNOB_1_FRONT: J15.18 (Pin_18), P1.2
- new net KNOB_2_FRONT: J15.19 (Pin_19), P2.2
- new net NEOPIXEL_DATA_FRONT: J15.23 (Pin_23), LED1.3 (DIN)
- new net OLED_CLK: J14.22 (Pin_22)
- new net OLED_DIN: J14.21 (Pin_21)
- new net OLED_D/C: J14.20 (Pin_20)
Other:
- note added: "PIN HEADERS"
- moved on the sheet: C25, R61, SW1, SW2, U7E, U9E

Commit message: kicad save
Parts:
- added C25, C26: 10u, Capacitor_SMD:C_0805_2012Metric, symbol Device:C_Polarized
- added C30: 100n, Capacitor_SMD:C_0402_1005Metric, symbol Device:C
- added D1, D2: ${SIM.PARAMS}, Diode_SMD:D_SMA, symbol Simulation_SPICE:DIODE
- added J9: Conn_02x05_Odd_Even, Eurorack:Eurorack Power Header, symbol Connector_Generic:Conn_02x05_Odd_Even
- U6: renamed from U5; footprint Package_TO_SOT_SMD:TO-252-3_TabPin4 -> Package_SO:SOIC-8_5.23x5.23mm_P1.27mm
- renumbered C9 to C10, C10 to C11, C11 to C12, C12 to C13, C13 to C14, C14 to C15, C15 to C16, C16 to C17, C17 to C18, C18 to C19, C19 to C20, C27 to C21, C28 to C22, C29 to C23, C30 to C24, C26 to C27, C20 to C28, C21 to C29, C22 to C31, C23 to C32, C25 to C33, C24 to C4, C4 to C5, C5 to C6, C6 to C7, C7 to C8, C8 to C9, D1 to D3, D2 to D4, J14 to J1, J3 to J10, J4 to J11, J5 to J12, J6 to J13, J7 to J14, J8 to J15, J13 to J16, J9 to J2, J11 to J3, J15 to J4, J1 to J5, J2 to J6, J12 to J7, J10 to J8, LED11 to LED10, LED10 to LED11, LED5 to LED2, LED2 to LED3, LED6 to LED4, LED3 to LED5, LED7 to LED6, LED4 to LED7, R9 to R10, R10 to R11, R11 to R12, R12 to R13, R13 to R14, R14 to R15, R47 to R16, R53 to R17, R15 to R18, R16 to R19, R17 to R20, R18 to R21, R48 to R22, R44 to R23, R54 to R24, R55 to R25, R19 to R26, R45 to R27, R56 to R28, R20 to R29, R46 to R3, R21 to R30, R22 to R31, R23 to R32, R24 to R33, R25 to R34, R57 to R35, R49 to R36, R26 to R37, R27 to R38, R58 to R39, R3 to R4, R59 to R40, R50 to R41, R51 to R42, R60 to R43, R52 to R44, R28 to R45, R29 to R46, R30 to R47, R31 to R48, R32 to R49, R4 to R5, R33 to R50, R34 to R51, R35 to R52, R36 to R53, R37 to R54, R38 to R55, R39 to R56, R40 to R57, R41 to R58, R61 to R59, R5 to R6, R42 to R60, R43 to R61, R6 to R7, R7 to R8, R8 to R9, SW3 to SW1, SW1 to SW2, SW2 to SW3, U8 to U10, U11 to U3, U3 to U4, U4 to U5, U6 to U7, U7 to U8
Connections:
- net +12V: now also C25.1, D1.2 (K)
- net +3.3V: now also C30.1
- net -12V: now also C26.2, D2.1 (A)
- net BUTTON_1: now also U4.13 (GPIO10)
- net BUTTON_2: now also U4.12 (GPIO9)
- net Earth: now also C25.2, C26.1, C30.2, J9.3 (Pin_3), J9.4 (Pin_4), J9.5 (Pin_5), J9.6 (Pin_6), J9.7 (Pin_7), J9.8 (Pin_8)
- net OLED_CLK: now also U4.17 (GPIO14)
- net OLED_DIN: now also U4.14 (GPIO11)
- net OLED_D/C: now also U4.16 (GPIO13)
- net USB_DM renamed USB_DN
- new net: D2.2 (K), J9.1 (Pin_1), J9.2 (Pin_2)
- new net: D1.1 (A), J9.10 (Pin_10), J9.9 (Pin_9)

Commit message: kicad save
Parts:
- removed J1: Conn_02x12_Counter_Clockwise, Connector_PinSocket_2.54mm:PinSocket_2x12_P2.54mm_Vertical, symbol Connector_Generic:Conn_02x12_Counter_Clockwise
- removed J4: Conn_02x12_Counter_Clockwise, Connector_PinHeader_2.54mm:PinHeader_2x12_P2.54mm_Vertical, symbol Connector_Generic:Conn_02x12_Counter_Clockwise
- removed J9: Conn_02x05_Odd_Even, Eurorack:Eurorack Power Header, symbol Connector_Generic:Conn_02x05_Odd_Even
- removed R16, R17, R35, R36: 10K, Resistor_SMD:R_0402_1005Metric, symbol Device:R
- removed R6, R7: 5K1, Resistor_SMD:R_0402_1005Metric, symbol Device:R
- removed SW1: BOOT, Button_Switch_THT:SW_PUSH_6mm_H4.3mm, symbol Switch:SW_Push
- removed USB1: USB_C_Receptacle_USB2.0, Connector_USB:USB_C_Receptacle_Amphenol_12401548E4-2A, symbol Connector:USB_C_Receptacle_USB2.0
- added C34: 10u, Capacitor_SMD:C_0805_2012Metric, symbol Device:C_Polarized
- added D5: ${SIM.PARAMS}, Diode_SMD:D_SMA, symbol Simulation_SPICE:DIODE
- added J17: Conn_02x08_Odd_Even, Eurorack:Eurorack Power Header 16 Pin, symbol Connector_Generic:Conn_02x08_Odd_Even
- added J18, J9: Conn_01x16_Pin, Connector_PinHeader_2.54mm:PinHeader_1x16_P2.54mm_Vertical, symbol Connector:Conn_01x16_Pin
- added J19, J4: Conn_01x16_Pin, Connector_PinSocket_2.54mm:PinSocket_1x16_P2.54mm_Vertical, symbol Connector:Conn_01x16_Pin
- added J20: Conn_01x06_Pin, Connector_PinHeader_2.54mm:PinHeader_1x06_P2.54mm_Horizontal, symbol Connector:Conn_01x06_Pin
- added TP1, TP2, TP3, TP4, TP5, TP6, TP7, TP8: TestPoint, TestPoint:TestPoint_Pad_1.0x1.0mm, symbol Connector:TestPoint
Connections:
- net +12V: now also TP2.1
- net +3.3V: now also J4.15 (Pin_15), TP5.1
- net +3.3V_FRONT: now also J9.15 (Pin_15)
- net +5V: now also C34.1, D5.2 (K), J20.1 (Pin_1), J4.16 (Pin_16), TP1.1
- net +5V_FRONT: now also J9.16 (Pin_16)
- net -10VREF: now also TP8.1
- net -12V: now also TP3.1
- net -2.048VREF: now also TP6.1
- net -4.096VREF: now also TP7.1
- net BUTTON_1: now also J4.13 (Pin_13)
- net BUTTON_1_FRONT: now also J9.13 (Pin_13)
- net BUTTON_2: now also J4.12 (Pin_12)
- net BUTTON_2_FRONT: now also J9.12 (Pin_12)
- net CV_INPUT_1: now also J4.6 (Pin_6); no longer R27.2, U10.1 (CH1+), U9.1
- net CV_INPUT_1_FRONT: now also J9.6 (Pin_6)
- net CV_INPUT_2: now also J4.7 (Pin_7); no longer R44.2, U10.3 (CH2+), U9.7
- net CV_INPUT_2_FRONT: now also J9.7 (Pin_7)
- net CV_INPUT_3: now also J4.8 (Pin_8); no longer R28.2, U10.11 (CH3+), U9.8
- net CV_INPUT_3_FRONT: now also J9.8 (Pin_8)
- net CV_INPUT_4: now also J4.9 (Pin_9); no longer R43.2, U10.13 (CH4+), U9.14
- net CV_INPUT_4_FRONT: now also J9.9 (Pin_9)
- net CV_OUTPUT_1: now also J19.2 (Pin_2)
- net CV_OUTPUT_1_FRONT: now also J18.2 (Pin_2)
- net CV_OUTPUT_2: now also J19.3 (Pin_3)
- net CV_OUTPUT_2_FRONT: now also J18.3 (Pin_3)
- net CV_OUTPUT_3: now also J19.4 (Pin_4)
- net CV_OUTPUT_3_FRONT: now also J18.4 (Pin_4)
- net CV_OUTPUT_4: now also J19.5 (Pin_5)
- net CV_OUTPUT_4_FRONT: now also J18.5 (Pin_5)
- net CV_OUTPUT_5: now also J19.6 (Pin_6)
- net CV_OUTPUT_5_FRONT: now also J18.6 (Pin_6)
- net CV_OUTPUT_6: now also J19.7 (Pin_7)
- net CV_OUTPUT_6_FRONT: now also J18.7 (Pin_7)
- net CV_OUTPUT_7: now also J19.8 (Pin_8)
- net CV_OUTPUT_7_FRONT: now also J18.8 (Pin_8)
- net CV_OUTPUT_8: now also J19.9 (Pin_9)
- net CV_OUTPUT_8_FRONT: now also J18.9 (Pin_9)
- net Earth: now also C33.2, R59.1, C34.2, J17.3 (Pin_3), J17.4 (Pin_4), J17.5 (Pin_5), J17.6 (Pin_6), J17.7 (Pin_7), J17.8 (Pin_8), J19.1 (Pin_1), J20.4 (Pin_4), J4.1 (Pin_1), J4.14 (Pin_14), J4.2 (Pin_2), J4.3 (Pin_3), J4.4 (Pin_4), J4.5 (Pin_5), TP4.1
- net GND_FRONT: now also J18.1 (Pin_1), J9.1 (Pin_1), J9.14 (Pin_14), J9.2 (Pin_2), J9.3 (Pin_3), J9.4 (Pin_4), J9.5 (Pin_5); no longer C33.2, R59.1
- net INPUT_DETECT: now also J19.10 (Pin_10)
- net INPUT_DETECT_FRONT: now also J2.2 (TN), J3.2 (TN), J7.2 (TN), J8.2 (TN), J18.10 (Pin_10)
- net IREF: now also J19.12 (Pin_12); no longer J16.26 (Pin_26)
- net KNOB_1: now also J4.11 (Pin_11)
- net KNOB_1_FRONT: now also J9.11 (Pin_11)
- net KNOB_2: now also J4.10 (Pin_10)
- net KNOB_2_FRONT: now also J9.10 (Pin_10)
- net NEOPIXEL_DATA: now also J19.11 (Pin_11)
- net NEOPIXEL_DATA_FRONT: now also J18.11 (Pin_11)
- net OLED_CLK: now also J19.14 (Pin_14)
- net OLED_CLK_FRONT: now also J18.14 (Pin_14)
- net OLED_DIN: now also J19.15 (Pin_15)
- net OLED_DIN_FRONT: now also J18.15 (Pin_15)
- net OLED_D/C: now also J19.16 (Pin_16)
- net OLED_D/C_FRONT: now also J18.16 (Pin_16)
- net RUN: now also J20.6 (Pin_6)
- net USB_DN: now also J20.2 (Pin_2)
- net USB_DP: now also J20.3 (Pin_3)
- net VCOMH: now also J19.13 (Pin_13); no longer J16.27 (Pin_27)
- net at C11.1, R12.1, R13.1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: now also U7.12 (+); no longer U7.3 (+)
- net at C20.1, R31.1, R32.1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: now also U8.3 (+); no longer U8.5 (+)
- net at C12.2, R19.1, R21.2: now also U8.14; no longer U8.1
- net at C12.1, R14.1, R15.1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: now also U8.12 (+); no longer U8.3 (+)
- net at C32.2, R58.1, R61.2: now also U8.8; no longer U8.14
- net at C32.1, R55.1, R56.1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: now also U8.10 (+); no longer U8.12 (+)
- net at C28.1, R45.1, R46.1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: now also U7.5 (+); no longer U7.10 (+)
- net at C28.2, R49.1, R51.2: now also U7.7; no longer U7.8
- net at C29.1, R47.1, R48.1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: now also U8.5 (+); no longer U8.10 (+)
- net at C29.2, R50.1, R52.2: now also U8.7; no longer U8.8
- net at C20.2, R34.1, R38.2: now also U8.1; no longer U8.7
- net at C11.2, R18.1, R20.2: now also U7.14; no longer U7.1
- net at D2.2 (K): now also J17.1 (Pin_1), J17.2 (Pin_2)
- net at D1.1 (A): now also J17.10 (Pin_10), J17.9 (Pin_9)
- net at C19.2, R33.1, R37.2: now also U7.1; no longer U7.7
- net at C19.1, R29.1, R30.1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: now also U7.3 (+); no longer U7.5 (+)
- net at C31.2, R57.1, R60.2: now also U7.8; no longer U7.14
- net at C31.1, R53.1, R54.1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: now also U7.10 (+); no longer U7.12 (+)
- net BOOTSEL: now reaches R11.2
- net BOOTSEL: now also J20.5 (Pin_5)
- net D2: no longer names the net of J16.20 (Pin_20)
- new net +5V_EURO: D5.1 (A), J17.11 (Pin_11), J17.12 (Pin_12)
- new net ADC_INPUT_1: R27.2, U10.1 (CH1+), U9.1
- new net ADC_INPUT_2: R44.2, U10.3 (CH2+), U9.7
- new net ADC_INPUT_3: R28.2, U10.11 (CH3+), U9.8
- new net ADC_INPUT_4: R43.2, U10.13 (CH4+), U9.14
- new net IREF_FRONT: J16.26 (Pin_26), J18.12 (Pin_12)
- new net VCOMH_FRONT: J16.27 (Pin_27), J18.13 (Pin_13)
- no-connect marks 17 -> 16
Other:
- moved on the sheet: C25, C26, C33, D1, D2, R59, U7A, U7B, U7C, U7D, U8A, U8B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

Commit message: kicad save
Parts:
- removed J20: Conn_01x06_Pin, Connector_PinHeader_2.54mm:PinHeader_1x06_P2.54mm_Horizontal, symbol Connector:Conn_01x06_Pin
- removed TP1, TP2, TP3, TP5: TestPoint, TestPoint:TestPoint_Pad_1.0x1.0mm, symbol Connector:TestPoint
- added C35, C36: 100n, Capacitor_SMD:C_0402_1005Metric, symbol Device:C
- added JUMPER1, JUMPER3: UNI/BIPOLAR, Connector_PinHeader_2.54mm:PinHeader_1x03_P2.54mm_Vertical, symbol Connector:Conn_01x03_Pin
- added P1: USB_C_Plug_USB2.0, Connector_USB:USB_C_Receptacle_G-Switch_GT-USB-7010ASV, symbol Connector:USB_C_Plug_USB2.0
- added R6, R7: 22, Resistor_SMD:R_0402_1005Metric, symbol Device:R
- added U11: L7805, Package_TO_SOT_SMD:TO-252-2, symbol Regulator_Linear:L7805
- J11: renamed from J17; footprint Eurorack:Eurorack Power Header 16 Pin -> Eurorack:Eurorack Power Header 16 Pin Unlabeled
- renumbered C34 to C28, C28 to C29, C29 to C30, C30 to C31, C31 to C32, C32 to C33, C33 to C34, J9 to J1, J8 to J10, J10 to J12, J11 to J13, J12 to J14, J13 to J15, J14 to J16, J15 to J17, J16 to J18, J18 to J2, J2 to J3, J3 to J4, J4 to J5, J5 to J6, J6 to J7, J19 to J8, J7 to J9, JUMPER1 to JUMPER2, P1 to P2, P2 to P3, R18 to R16, R19 to R17, R20 to R18, R21 to R19, R22 to R20, R23 to R21, R24 to R22, R25 to R23, R26 to R24, R27 to R25, R28 to R26, R29 to R27, R30 to R28, R31 to R29, R32 to R30, R33 to R31, R34 to R32, R37 to R33, R38 to R34, R39 to R35, R40 to R36, R41 to R37, R42 to R38, R43 to R39, R44 to R40, R45 to R41, R46 to R42, R47 to R43, R48 to R44, R49 to R45, R50 to R46, R51 to R47, R52 to R48, R53 to R49, R54 to R50, R55 to R51, R56 to R52, R57 to R53, R58 to R54, R59 to R55, R60 to R56, R61 to R57, SW2 to SW1, SW3 to SW2
Connections:
- net +12V: now also TP7.1, JUMPER3.3 (Pin_3)
- net +5V: now also TP6.1, C36.1, P1.A4 (VBUS), P1.A9 (VBUS), P1.B4 (VBUS), P1.B9 (VBUS), U11.3 (OUT)
- net -10VREF: no longer TP8.1
- net -12V: now also TP8.1
- net -2.048VREF: no longer TP6.1
- net -4.096VREF: no longer TP7.1
- net BOOTSEL: now also JUMPER1.3 (Pin_3)
- net Earth: now also C35.2, C36.2, JUMPER1.2 (Pin_2), P1.A1 (GND), P1.A12 (GND), P1.B1 (GND), P1.B12 (GND), U11.2 (GND)
- net RUN: now also JUMPER1.1 (Pin_1)
- net USB_DN: now also R6.2
- net USB_DP: now also R7.2
- new net: P1.A6 (D+), R7.1
- new net: P1.A7 (D-), R6.1
- new net 5VREG_INPUT: C35.1, JUMPER3.2 (Pin_2), U11.1 (IN)
- no-connect marks 16 -> 18
Other:
- note added: "Jumper sets internal 5V regulator"
