File: hardware/EuroPi-X/kicad/EuroPi-X.kicad_sch (KiCad schematic)
At the start: 156 parts, among them J1 Conn_01x16_Pin, J10 Thonkiconn_Mono_Jack, J11 Conn_02x08_Odd_Even, J12 Thonkiconn_Mono_Jack, J13 Thonkiconn_Mono_Jack, J14 Thonkiconn_Mono_Jack, J15 Thonkiconn_Mono_Jack, J16 Thonkiconn_Mono_Jack, J17 Thonkiconn_Mono_Jack, J18 Conn_01x30_Pin, J19 Conn_01x04_Pin, J2 Conn_01x16_Pin, J20 Conn_01x04_Pin, J21 Conn_01x04_Pin, J3 Thonkiconn_Mono_Jack, J4 Thonkiconn_Mono_Jack, J5 Conn_01x16_Pin, J6 Thonkiconn_Mono_Jack, J7 Thonkiconn_Mono_Jack, J8 Conn_01x16_Pin, J9 Thonkiconn_Mono_Jack, P1 USB_C_Plug_USB2.0, P2 Potentiometer_9mm_Vertical_Li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, P3 Potentiometer_9mm_Vertical_Li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, Q1 BSS138, SW1 B1, SW2 B2, U1 LM4030-4.096, U10 MCP3428, U11 L7805, U2 LM4040DBZ-2.0, U3 LM4040DBZ-10, U4 RP2040, U7 TL074, U8 TL074, U9 MCP6004, Y1 Crystal_GND2

Commit message: save and export
Parts:
- removed C18, C34: 100n, Capacitor_SMD:C_0402_1005Metric, symbol Device:C
- removed J18: Conn_01x30_Pin, Connector_FFC-FPC:Hirose_FH41-30S-0.5SH_1x30_1MP_1SH_P0.5mm_Horizontal, symbol Connector:Conn_01x30_Pin
- removed J19, J21: Conn_01x04_Pin, Connector_PinHeader_2.54mm:PinHeader_1x04_P2.54mm_Vertical, symbol Connector:Conn_01x04_Pin
- removed J20: Conn_01x04_Pin, Connector_JST:JST_SH_SM04B-SRSS-TB_1x04-1MP_P1.00mm_Horizontal, symbol Connector:Conn_01x04_Pin
- removed JUMPER1, JUMPER2: UNI/BIPOLAR, Connector_PinHeader_2.54mm:PinHeader_1x03_P2.54mm_Vertical, symbol Connector:Conn_01x03_Pin
- removed R55: ~, Resistor_SMD:R_0402_1005Metric, symbol Device:R
- removed U1: LM4030-4.096, Package_TO_SOT_SMD:SOT-23-5, symbol Reference_Voltage:LM4030-4.096
- added C37, C38, C39, C40, C41: 100n, Capacitor_SMD:C_0402_1005Metric, symbol Device:C
- added J20: Conn_01x06_Pin, Connector_PinHeader_2.54mm:PinHeader_1x06_P2.54mm_Vertical, symbol Connector:Conn_01x06_Pin
- added J22: Conn_01x11_Pin, Connector_PinHeader_2.54mm:PinHeader_1x11_P2.54mm_Vertical, symbol Connector:Conn_01x11_Pin
- added OLED1: ~, Eurorack:Enoki OLED SSD1306 128x64, symbol Eurorack:Enoki_OLED_SSD1306_128x64
- added R60: 200R, Resistor_SMD:R_0402_1005Metric, symbol Device:R
- added SW3: ~, Eurorack:TS-1187A-B-A-B, symbol Eurorack:Tactile_Switch_
- added U12: LM4040DBZ-4.1, Package_TO_SOT_SMD:SOT-23, symbol Reference_Voltage:LM4040DBZ-4.1
- C1, C16: value 1u -> 100n; JLC (none) -> C1525; JLCPCB PART# C52923 -> (none)
- C10, C2, C3, C4, C7: JLC (none) -> C52923; JLCPCB PART# C52923 -> (none)
- C11, C12, C19, C20, C29, C30, C32, C33: JLC (none) -> C1546
- C13, C17: value 100n -> 2u2; JLC (none) -> C12530; JLCPCB PART# C1525 -> (none)
- C14, C21, C22, C23, C24, C27, C31, C35, C36, C5, C6: JLC (none) -> C1525; JLCPCB PART# C1525 -> (none)
- C15: value 1u -> 2u2; JLC (none) -> C12530; JLCPCB PART# C52923 -> (none)
- C25, C26, C28: JLC (none) -> C15850; JLCPCB PART# C15850 -> (none)
- C8, C9: JLC (none) -> C32949; JLCPCB PART# C32949 -> (none)
- D1, D2, D5: JLC (none) -> C95872; JLCPCB PART# C95872 -> (none)
- D3, D4, D6: footprint Diode_SMD:D_0402_1005Metric -> Diode_SMD:D_SOD-123; JLC (none) -> C8598
- DAC1, DAC2: JLC (none) -> C478093; JLCPCB PART# C108207 -> (none)
- P1: JLC (none) -> C309361; JLCPCB PART# C309361 -> (none)
- Q1: JLC (none) -> C112239; JLCPCB PART# C112239 -> (none)
- R1, R2, R3: JLC (none) -> C25879
- R10, R6, R7, R8, R9: JLC (none) -> C25744; JLCPCB PART# C25744 -> (none)
- R11, R18, R19, R33, R34, R47, R48, R56, R57: JLC (none) -> C11702; JLCPCB PART# C11702 -> (none)
- R12, R13, R14, R15, R20, R21, R22, R23, R27, R28, R29, R30, R35, R36, R37, R38, R41, R42, R43, R44, R49, R50, R51, R52: JLC (none) -> C25741; JLCPCB PART# C25741 -> (none)
- R16, R17, R31, R32, R45, R46, R53, R54: JLC (none) -> C170277; JLCPCB PART# C170277 -> (none)
- R24: value 27R4 -> 1R; JLC (none) -> C25086
- R25, R26, R39, R40: JLC (none) -> C25756; JLCPCB PART# C25756 -> (none)
- R4, R5: JLC (none) -> C25100
- R58: JLC (none) -> C25092; JLCPCB PART# C25092 -> (none)
- R59: JLC (none) -> C25744; JLCPCB PART# C25092 -> (none)
- U10: JLC (none) -> C560166; JLCPCB PART# C560166 -> (none)
- U11: footprint Package_TO_SOT_SMD:TO-252-3_TabPin2 -> Package_TO_SOT_SMD:TO-252-2; JLC (none) -> C58069
- U2: JLC (none) -> C144273
- U3: JLC (none) -> C129969
- U4: JLC (none) -> C2040; JLCPCB PART# C2040 -> (none)
- U5: footprint Package_TO_SOT_SMD:TO-252-3_TabPin4 -> Package_TO_SOT_SMD:SOT-23-3; JLC (none) -> C5446
- U6: JLC (none) -> C2940195
- U7, U8: footprint Package_SO:SOIC-16_3.9x9.9mm_P1.27mm -> Package_SO:SOIC-14_3.9x8.7mm_P1.27mm; JLC (none) -> C6963
- U9: JLC (none) -> C50282
- Y1: JLC (none) -> C9002; JLCPCB PART# C9002 -> (none)
Connections:
- net IREF is gone; now on net I2C0_SDA: J8.12 (Pin_12)
- net OLED_CLK_FRONT is gone; now on net GND_FRONT: J2.14 (Pin_14)
- net OLED_DIN_FRONT is gone; now on net GND_FRONT: J2.15 (Pin_15)
- net OLED_D/C_FRONT is gone; now on net GND_FRONT: J2.16 (Pin_16)
- net VCOMH is gone; now on net I2C0_SCL: J8.13 (Pin_13)
- net +12V: now also J20.6 (Pin_6)
- net +3.3V: now also C1.1, C15.1, C5.1, C6.1, C37.1, C38.1, C39.1, C40.1, J22.5 (Pin_5), J22.9 (Pin_9), R60.2; no longer C16.1, C17.1, R24.1, U4.48 (USB_VDD)
- net +3.3V_FRONT: now also OLED1.8 (3V3)
- net -2.048VREF: now also J20.3 (Pin_3)
- net -4.096VREF: now also J20.1 (Pin_1), U12.2 (A)
- net 5VREG_INPUT: now also J20.5 (Pin_5)
- net ADC_VDD: no longer C13.1, C15.1, R24.2
- net BOOTSEL: now also J22.7 (Pin_7), SW3.1 (A)
- net DAC_OFFSET: now also J20.2 (Pin_2)
- net Earth: now also J8.14 (Pin_14), J8.15 (Pin_15), J8.16 (Pin_16), C37.2, C38.2, C39.2, C40.2, C41.2, J22.2 (Pin_2), J22.4 (Pin_4), J22.8 (Pin_8), SW3.3 (C), U12.1 (K)
- net GND_FRONT: now also OLED1.7 (GND)
- net I2C1_SCL: now also J22.11 (Pin_11)
- net I2C1_SDA: now also J22.10 (Pin_10)
- net INPUT_DETECT: now also U4.15 (GPIO12); no longer U4.18 (GPIO15)
- net NEOPIXEL_DATA_3V3: now also U4.14 (GPIO11); no longer U4.17 (GPIO14)
- net OUTPUT_MODE: now also U4.13 (GPIO10); no longer U4.15 (GPIO12)
- net RUN: now also J22.6 (Pin_6)
- net SWCLK: now also J22.1 (Pin_1)
- net SWDIO: now also J22.3 (Pin_3)
- net USB_DETECT: now also U4.36 (GPIO24)
- net +1V1: now reaches U4.23 (DVDD), U4.45 (VREG_VOUT), U4.50 (DVDD)
- net +1V1: now also C13.1, C16.1, C41.1; no longer C1.1, C5.1, C6.1
- net IREF_FRONT renamed I2C0_SDA_FRONT
- net I2C0_SDA_FRONT: now also OLED1.5 (SDA)
- removed net OLED_CLK: J8.14 (Pin_14), U4.13 (GPIO10)
- removed net OLED_DIN: J8.15 (Pin_15), U4.14 (GPIO11)
- net OLED_D/C: no longer names the net of U4.16 (GPIO13)
- net OLED_D/C: no longer J8.16 (Pin_16)
- net VCOMH_FRONT renamed I2C0_SCL_FRONT
- net I2C0_SCL_FRONT: now also OLED1.6 (SCK)
- new net ADC_ADVDD: C17.1, R24.1
- new net ADC_VREF: R24.2, R60.1
- new net USB_VDD: U4.48 (USB_VDD)
- no-connect marks 30 -> 27
Other:
- note added: "PIN01"
- note added: "PIN10"
- note added: "PIN22"
- note added: "PIN23"
- note added: "PIN33"
- note added: "PIN42"
- note added: "PIN43"
- note added: "PIN44"
- note added: "PIN45"
- note added: "PIN49"
- note added: "PIN50"
- note added: "The Toadstool Tech Enoki board is used for the OLED as it has a small enough board outline to fit on the front PCB. It is used in i2c mode so the on-board solder jumpers must be bridged. The SPI pins are left unconnected, and the two support headers are soldered but are not connected to any signal"
- note added: "The male header (above) is used on the front PCB and the female header (below) is used on the back PCB. This is so that in the event the standoff fails or is improperly tightened and the PCBs pull apart in the rack, the power rails that are routed through the headers are not exposed via the male pins so can't cause damage to the circuit or power supply if they contact other modules or metal in th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"
- note added: "i2c bus 1 of the RP2040"
- note removed: "2.54mm connector for i2c"
- note removed: "Expander for buttons (reset and bootsel)"
- note removed: "STEMMA QT connector for i2c"
- note removed: "i2c connectors use i2c bus 1"
- moved on the sheet: C10, C11, C12, C14, C19, C2, C20, C21, C22, C23, C24, C25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

Commit message: neaten schematic and annotate more
Other:
- note added: "Crystal"
- note added: "Flash"
- note added: "NEOPIXEL RGB LEDS"
- note added: "Serial Wire Debug"
- note added: "The DACs have a programmable gain which is set to output 0-4.096V. The channel must also be set to 1 in code to use the internal 2.048V reference"
- moved on the sheet: C10, C35, C36, C7, J10, J3, J4, R20, R21, R22, R23, R25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

Commit message: save
Parts:
- P1: JLC C309361 -> C2927037
Changed lines of the file:
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@@
       (effects (font (size 1.27 1.27)) hide)
     )
-    (property "JLC" "C309361" (at 82.55 72.39 0)
+    (property "JLC" "C2927037" (at 82.55 72.39 0)
       (effects (font (size 1.27 1.27)) hide)
     )

Commit message: save
Parts:
- removed J20: Conn_01x06_Pin, Connector_PinHeader_2.54mm:PinHeader_1x06_P2.54mm_Vertical, symbol Connector:Conn_01x06_Pin
- added C18: 100n, Capacitor_SMD:C_0402_1005Metric, symbol Device:C
- added J18: Conn_01x03_Pin, Connector_PinHeader_2.54mm:PinHeader_1x03_P2.54mm_Vertical, symbol Connector:Conn_01x03_Pin
- added R55, R61: 270K, Resistor_SMD:R_0402_1005Metric, symbol Device:R
- added SW4, SW5: ~, Package_TO_SOT_SMD:SOT-363_SC-70-6, symbol Eurorack:WAS3157B
- added U1: MCP6002-xSN, Package_SO:SOIC-8_3.9x4.9mm_P1.27mm, symbol Amplifier_Operational:MCP6002-xSN
- R8, R9: value 10K -> 270K; JLC C25744 -> C170277
Connections:
- net +12V: now also J5.1 (Pin_1), R1.2, R2.2, J18.3 (Pin_3)
- net +5V: now also C18.1, SW4.5 (VCC), SW5.5 (VCC), U1.8 (V+)
- net -12V: now also J5.2 (Pin_2); no longer R1.2, R2.2
- net 5VREG_INPUT: now also J18.2 (Pin_2)
- net Earth: now also C18.2, SW4.2 (GND), SW5.2 (GND), U1.3 (+), U1.4 (V-), U1.6 (-); no longer J5.1 (Pin_1), J5.2 (Pin_2), R9.1
- net GND_FRONT: no longer J1.1 (Pin_1), J1.2 (Pin_2)
- net INPUT_DETECT: now also U4.16 (GPIO13); no longer U4.15 (GPIO12)
- net NEOPIXEL_DATA_3V3: now also U4.15 (GPIO12); no longer U4.14 (GPIO11)
- net -2.048VREF renamed +2.048VREF
- net +2.048VREF: now also SW4.1 (B1), SW5.1 (B1)
- net -4.096VREF renamed +4.096VREF
- net +4.096VREF: now also SW4.3 (B0), SW5.3 (B0)
- removed net DAC_OFFSET: R12.2, R14.2, R27.2, R29.2, R41.2, R43.2, R49.2, R51.2, R8.2
- net OUTPUT_MODE: no longer names the net of R8.1, R9.2
- net OUTPUT_MODE: now also U1.2 (-); no longer U4.13 (GPIO10)
- new net: R55.1, R61.2, U1.5 (+)
- new net DAC_1_OFFSET: R12.2, R27.2, R41.2, R49.2, R9.1, U1.1
- new net DAC_1_OFFSET_INVERTED: R8.2, SW4.4 (A)
- new net DAC_1_OUTPUT_MODE: SW4.6 (SEL), U4.13 (GPIO10)
- new net DAC_2_OFFSET: R14.2, R29.2, R43.2, R51.2, R61.1, U1.7
- new net DAC_2_OFFSET_INVERTED: R55.2, SW5.4 (A)
- new net DAC_2_OUTPUT_MODE: SW5.6 (SEL), U4.14 (GPIO11)
- no-connect marks 27 -> 28
Other:
- note added: "+2.048V REFERENCE"
- note added: "+4.096V REFERENCE"
- note added: "Despite being powered by a higher level (+5V), the WAS3157B analog switch has a threshold of only 1.8V for logic"
- note added: "OUTPUT_MODE is a digital signal from the RP2040 that can be set in code to determine the polarity of the outputs: 0 - unipolar 0-10V 1 - bipolar ±5V"
- note added: "The signal is split on the PCB into two nets - CV_OUTPUT_X is on the back PCB, and CV_OUTPUT_X_FRONT PCB. Once the module is assembled, these nets are connected by the 2.54mm headers"
- note added: "The voltage references are kept positive (>0V) so that a more standard analog switch can be used. They are inverted before use in the output stage"
- note removed: "-2.048 is bipolar"
- note removed: "-2.048V REFERENCE"
- note removed: "-4.096V REFERENCE"
- note removed: "-4.096V is unipolar"
- note removed: "DAC_OFFSET is voltage divided down to 1.024V in bipolar mode, below the ~1.8V threshold for a GPIO to be read as 'high', or 2.048V in unipolar mode, above the threshold. Thus OUTPUT_MODE can be used by the software to determine if the module is in unipolar or bipolar mode without requiring an extra jumper"
- note removed: "Jumper sets output mode"
- moved on the sheet: Q1, R4, R5, R6, R7, U4

Commit message: save
Other:
- note added: "Although the 12V rails are not used on the front panel, they are included on this header for testing purposes"
- note added: "Despite being on the same pin header, multiple power and ground pins are included so that separate 2.54mm cables can be used to route the i2c, swd, and run/bootsel groups individually"
- note added: "The internal +3.3V regulator is used to generate the supply for the RP2040, which is also used for the buttons and knobs"
- note added: "The internal +5V regulator is only used if the jumper on the back of the PCB is set to 'no 5V rail' This allows users with a 5V rail to use the likely more powerful +5V regulator in the eurorack supply, thus reducing the strain on the +12V rail and reducing noise by separating analogue and digital supplies"
- moved on the sheet: C10, C35, C36, C7, U11, U5

Commit message: save
Other:
- note added: "-4.096V or -2.048V depending on OUTPUT_MODE setting"
- note added: "The DAC_X_OFFSET signals are inverted to make them negative for use in the DAC output circuit"
- note added: "The Neopixel LEDs are serial controlled, meaning only a single pin of the RP2040 is connected to the first LED, and the remaning LEDs are connected in series. They are powered by 5V, but the RP2040 signal is only 3.3V, so a BSS138 MOSFET is used as a level shifter"
- note removed: "The Neopixel LEDs are serial controlled, meaning only a single pin of the RP2040 is connected to the first LED, and the remaning LEDs are connected in series. They are powered by 5V, but the RP2040 signal is only 3.3V, so a level shifter is used."
Changed lines of the file:
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@@
+    (effects (font (size 1.27 1.27)) (justify left bottom))
+  )
+  (text "The DAC_X_OFFSET signals\nare inverted to make them\nnegative for use in the\nDAC output circuit"
+    (at 143.51 476.25 0)
     (effects (font (size 1.27 1.27)) (justify left bottom))
   )
@@
     (effects (font (size 1.27 1.27)) (justify left bottom))
   )
+  (text "-4.096V or\n-2.048V\ndepending on\nOUTPUT_MODE\nsetting"
+    (at 207.01 472.44 0)
+    (effects (font (size 1.27 1.27)) (justify left bottom))
+  )
   (text "PIN10" (at 342.9 163.83 0)
     (effects (font (size 1.27 1.27)) (justify left bottom))
@@
     (effects (font (size 1.27 1.27)) (justify left bottom))
   )
-  (text "The Neopixel LEDs are serial controlled, meaning only a single\npin of the RP2040 is connected to the first LED, and the remaning\nLEDs are connected in series.\n\nThey are powered by 5V, but the \nRP2040 signal is only 3.3V, so a level shifter is used."
-    (at 518.16 95.25 0)
+  (text "The Neopixel LEDs are serial controlled, meaning only a single\npin of the RP2040 is connected to the first LED, and the remaning\nLEDs are connected in series.\n\nThey are powered by 5V, but the \nRP2040 signal is only 3.3V, so a\nBSS138 MOSFET is used as a\nlevel shifter"
+    (at 518.16 107.95 0)
     (effects (font (size 1.27 1.27)) (justify left bottom))
   )
@@
     (effects (font (size 1.27 1.27)) (justify left bottom))
   )
-  (label "DAC_1_OFFSET" (at 358.14 389.89 180) (fields_autoplaced)
-    (effects (font (size 1.27 1.27)) (justify right bottom))
-  )
   (label "DAC_2_OFFSET" (at 269.24 449.58 180) (fields_autoplaced)

Commit message: add falstad sim links
Other:
- note added: "If a signal did go above the range of ±10V, it would still be clamped to the rails of the op-amp, which are 0V and +3.3V, so the ADC input is protected for any input"
- note added: "Input stage Falstad simulation: https://tinyurl.com/24wc45cd"
- note added: "It has the offset of -10V added to it, resulting in a range of -20V to 0V"
- note added: "It is then inverted and attenuated by 0.15x resulting in a range of +3V to 0V, which is a safe range to feed into the +3.3V tolerant ADC input."
- note added: "Output stage Falstad simulation: https://tinyurl.com/2dm6q32a"
- note added: "The incoming signal is in the range ±10V"
- note added: "The signal is split on the PCB into two nets: CV_OUTPUT_X is on the back PCB, and CV_OUTPUT_X_FRONT is on the front PCB Once the module is assembled, these nets are connected through the 2.54mm headers"
- note removed: "The incoming signal is in the range ±10V It has the offset of -10V added to it, resulting in a range of -20V to 0V It is then inverted and attenuated by 0.15x resulting in a range of +3V to 0V, which is a safe range to feed into the +3.3V tolerant ADC input. If a signal did go above the range of ±10V, it would still be clamped to the rails of the op-amp, which are 0V and +3.3V, so the ADC input i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"
- note removed: "The signal is split on the PCB into two nets - CV_OUTPUT_X is on the back PCB, and CV_OUTPUT_X_FRONT PCB. Once the module is assembled, these nets are connected by the 2.54mm headers"
- moved on the sheet: J10, J3, J4, J9, R20, R21, R22, R23, R25, R26, R35, R36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

Commit message: save
Parts:
- added NT1: NetTie_2, NetTie:NetTie-2_SMD_Pad0.5mm, symbol Device:NetTie_2
Connections:
- net GND_FRONT: now also NT1.2; no longer J1.5 (Pin_5), P2.1, P3.1
- new net AGND_FRONT: J1.5 (Pin_5), NT1.1, P2.1, P3.1
Changed lines of the file:
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@@
   (junction (at 725.17 480.06) (diameter 0) (color 0 0 0 0)
   )
-  (junction (at 675.64 355.6) (diameter 0) (color 0 0 0 0)
-  )
   (junction (at 491.49 414.02) (diameter 0) (color 0 0 0 0)
   )
@@
   (junction (at 351.79 171.45) (diameter 0) (color 0 0 0 0)
   )
-  (junction (at 308.61 449.58) (diameter 0) (color 0 0 0 0)
+  (junction (at 678.18 355.6) (diameter 0) (color 0 0 0 0)
+  )
+  (junction (at 678.18 452.12) (diameter 0) (color 0 0 0 0)
   )
-  (junction (at 675.64 358.14) (diameter 0) (color 0 0 0 0)
+  (junction (at 308.61 449.58) (diameter 0) (color 0 0 0 0)
   )
   (junction (at 91.44 429.26) (diameter 0) (color 0 0 0 0)
@@
   (junction (at 232.41 161.29) (diameter 0) (color 0 0 0 0)
   )
-  (junction (at 678.18 452.12) (diameter 0) (color 0 0 0 0)
-  )
   (junction (at 491.49 449.58) (diameter 0) (color 0 0 0 0)
   )
@@
   (junction (at 113.03 383.54) (diameter 0) (color 0 0 0 0)
   )
-  (junction (at 678.18 454.66) (diameter 0) (color 0 0 0 0)
-  )
   (junction (at 582.93 463.55) (diameter 0) (color 0 0 0 0)
   )
@@
     (stroke (width 0) (type default))
   )
+  (wire (pts (xy 678.18 358.14) (xy 678.18 355.6))
+    (stroke (width 0) (type default))
+  )
   (wire (pts (xy 419.1 403.86) (xy 419.1 414.02))
     (stroke (width 0) (type default))
@@
     (stroke (width 0) (type default))
   )
+  (wire (pts (xy 675.64 358.14) (xy 678.18 358.14))
+    (stroke (width 0) (type default))
+  )
   (wire (pts (xy 373.38 449.58) (xy 377.19 449.58))
     (stroke (width 0) (type default))
@@
     (stroke (width 0) (type default))
   )
+  (wire (pts (xy 678.18 452.12) (xy 678.18 454.66))
+    (stroke (width 0) (type default))
+  )
   (wire (pts (xy 91.44 393.7) (xy 91.44 397.51))
     (stroke (width 0) (type default))
@@
     (stroke (width 0) (type default))
   )
-  (wire (pts (xy 680.72 355.6) (xy 675.64 355.6))
+  (wire (pts (xy 680.72 355.6) (xy 678.18 355.6))
     (stroke (width 0) (type default))
   )
@@
     (stroke (width 0) (type default))
   )
-  (wire (pts (xy 680.72 454.66) (xy 678.18 454.66))
+  (wire (pts (xy 689.61 341.63) (xy 698.5 341.63))
+    (stroke (width 0) (type default))
+  )
+  (wire (pts (xy 680.72 452.12) (xy 678.18 452.12))
     (stroke (width 0) (type default))
   )
@@
     (stroke (width 0) (type default))
   )
-  (wire (pts (xy 675.64 355.6) (xy 675.64 358.14))
+  (wire (pts (xy 709.93 341.63) (xy 703.58 341.63))
     (stroke (width 0) (type default))
   )
@@
     (stroke (width 0) (type default))
   )
+  (wire (pts (xy 675.64 360.68) (xy 680.72 360.68))
+    (stroke (width 0) (type default))
+  )
   (wire (pts (xy 247.65 290.83) (xy 237.49 290.83))
     (stroke (width 0) (type default))
@@
     (stroke (width 0) (type default))
   )
+  (wire (pts (xy 678.18 355.6) (xy 675.64 355.6))
+    (stroke (width 0) (type default))
+  )
   (wire (pts (xy 725.17 363.22) (xy 732.79 363.22))
     (stroke (width 0) (type default))
@@
     (stroke (width 0) (type default))
   )
-  (wire (pts (xy 675.64 358.14) (xy 675.64 360.68))
-    (stroke (width 0) (type default))
-  )
   (wire (pts (xy 452.12 449.58) (xy 457.2 449.58))
     (stroke (width 0) (type default))
@@
     (stroke (width 0) (type default))
   )
-  (wire (pts (xy 678.18 452.12) (xy 678.18 454.66))
-    (stroke (width 0) (type default))
-  )
   (wire (pts (xy 416.56 469.9) (xy 416.56 466.09))
     (stroke (width 0) (type default))
@@
     (effects (font (size 1.27 1.27)) (justify left bottom))
   )
+  (label "AGND_FRONT" (at 680.72 360.68 0) (fields_autoplaced)
+    (effects (font (size 1.27 1.27)) (justify left bottom))
+  )
   (label "CV_OUTPUT_8_FRONT" (at 725.17 370.84 180) (fields_autoplaced)
     (effects (font (size 1.27 1.27)) (justify right bottom))
@@
     (effects (font (size 1.27 1.27)) (justify left bottom))
   )
+  (label "GND_FRONT" (at 709.93 341.63 0) (fields_autoplaced)
+    (effects (font (size 1.27 1.27)) (justify left bottom))
+  )
   (label "I2C1_SDA" (at 113.03 140.97 0) (fields_autoplaced)
     (effects (font (size 1.27 1.27)) (justify left bottom))
@@
     (effects (font (size 1.27 1.27)) (justify left bottom))
   )
+  (label "AGND_FRONT" (at 566.42 316.23 180) (fields_autoplaced)
+    (effects (font (size 1.27 1.27)) (justify right bottom))
+  )
   (label "DAC_1_OUTC" (at 119.38 353.06 0) (fields_autoplaced)
     (effects (font (size 1.27 1.27)) (justify left bottom))
@@
     (effects (font (size 1.27 1.27)) (justify right bottom))
   )
+  (label "AGND_FRONT" (at 566.42 292.1 180) (fields_autoplaced)
+    (effects (font (size 1.27 1.27)) (justify right bottom))
+  )
   (label "CV_OUTPUT_6" (at 416.56 453.39 90) (fields_autoplaced)
     (effects (font (size 1.27 1.27)) (justify left bottom))
@@
     (effects (font (size 1.27 1.27)) (justify right bottom))
   )
-  (label "GND_FRONT" (at 566.42 292.1 180) (fields_autoplaced)
-    (effects (font (size 1.27 1.27)) (justify right bottom))
-  )
   (label "+5V_EURO" (at 706.12 289.56 180) (fields_autoplaced)
     (effects (font (size 1.27 1.27)) (justify right bottom))
@@
     (effects (font (size 1.27 1.27)) (justify left bottom))
   )
+  (label "AGND_FRONT" (at 689.61 341.63 180) (fields_autoplaced)
+    (effects (font (size 1.27 1.27)) (justify right bottom))
+  )
   (label "-10VREF" (at 340.36 285.75 180) (fields_autoplaced)
     (effects (font (size 1.27 1.27)) (justify right bottom))
@@
     (effects (font (size 1.27 1.27)) (justify right bottom))
   )
-  (label "GND_FRONT" (at 566.42 316.23 180) (fields_autoplaced)
-    (effects (font (size 1.27 1.27)) (justify right bottom))
-  )
   (label "GND_FRONT" (at 655.32 213.36 180) (fields_autoplaced)
     (effects (font (size 1.27 1.27)) (justify right bottom))
@@
     )
   )
+  (symbol (lib_id "Device:NetTie_2") (at 701.04 341.63 0) (unit 1)
+    (in_bom no) (on_board yes) (dnp no) (fields_autoplaced)
+    (property "Reference" "NT1" (at 701.04 337.82 0)
+      (effects (font (size 1.27 1.27)))
+    )
+    (property "Value" "NetTie_2" (at 701.04 340.36 0)
+      (effects (font (size 1.27 1.27)))
+    )
+    (property "Footprint" "NetTie:NetTie-2_SMD_Pad0.5mm" (at 701.04 341.63 0)
+      (effects (font (size 1.27 1.27)) hide)
+    )
+    (property "Datasheet" "~" (at 701.04 341.63 0)
+      (effects (font (size 1.27 1.27)) hide)
+    )
+    (pin "1")
+    (pin "2")
+    (instances
+      (project "EuroPi-X"
+        (path "/a1be51f2-61d0-4240-8665-f31cc7b044f7"
+          (reference "NT1") (unit 1)
+        )
+      )
+    )
+  )
   (symbol (lib_id "power:Earth") (at 434.34 91.44 90) (unit 1)
     (in_bom yes) (on_board yes) (dnp no) (fields_autoplaced)
@@
     )
   )
-  (symbol (lib_id "power:Earth") (at 680.72 454.66 90) (unit 1)
+  (symbol (lib_id "power:Earth") (at 680.72 452.12 90) (unit 1)
     (in_bom yes) (on_board yes) (dnp no) (fields_autoplaced)
-    (property "Reference" "#PWR028" (at 687.07 454.66 0)
+    (property "Reference" "#PWR028" (at 687.07 452.12 0)
       (effects (font (size 1.27 1.27)) hide)
     )
-    (property "Value" "Earth" (at 684.53 454.66 0)
+    (property "Value" "Earth" (at 684.53 452.12 0)
       (effects (font (size 1.27 1.27)) hide)
     )
-    (property "Footprint" "" (at 680.72 454.66 0)
+    (property "Footprint" "" (at 680.72 452.12 0)
       (effects (font (size 1.27 1.27)) hide)
     )
-    (property "Datasheet" "~" (at 680.72 454.66 0)
+    (property "Datasheet" "~" (at 680.72 452.12 0)
       (effects (font (size 1.27 1.27)) hide)
     )
