File: hardware/EuroPi-X/kicad/EuroPi-X.kicad_sch (KiCad schematic)
At the start: 164 parts, among them J1 Conn_01x16_Pin, J10 Thonkiconn_Mono_Jack, J11 Conn_02x08_Odd_Even, J12 Thonkiconn_Mono_Jack, J13 Thonkiconn_Mono_Jack, J14 Thonkiconn_Mono_Jack, J15 Thonkiconn_Mono_Jack, J16 Thonkiconn_Mono_Jack, J17 Thonkiconn_Mono_Jack, J18 Conn_01x03_Pin, J2 Conn_01x16_Pin, J22 Conn_01x11_Pin, J3 Thonkiconn_Mono_Jack, J4 Thonkiconn_Mono_Jack, J5 Conn_01x16_Pin, J6 Thonkiconn_Mono_Jack, J7 Thonkiconn_Mono_Jack, J8 Conn_01x16_Pin, J9 Thonkiconn_Mono_Jack, P1 USB_C_Plug_USB2.0, P2 Potentiometer_9mm_Vertical_Li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, P3 Potentiometer_9mm_Vertical_Li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, Q1 BSS138, SW1 B1, SW2 B2, U1 MCP6002-xSN, U10 MCP3428, U11 L7805, U12 LM4040DBZ-4.1, U2 LM4040DBZ-2.0, U3 LM4040DBZ-10, U4 RP2040, U7 TL074, U8 TL074, U9 MCP6004, Y1 Crystal_GND2

Commit message: save
Parts:
- SW4, SW5: JLC (none) -> C213161; JLC Rotation Offset (none) -> 270
- U1, U7, U8, U9: JLC Rotation Offset (none) -> 270
- U12, U2, U3, U5: JLC Rotation Offset (none) -> 180
Changed lines of the file:
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@@
       (effects (font (size 1.27 1.27)) hide)
     )
+    (property "JLC Rotation Offset" "180" (at 91.44 435.61 90)
+      (effects (font (size 1.27 1.27)) hide)
+    )
     (pin "1")
     (pin "2")
@@
       (effects (font (size 1.27 1.27)) hide)
     )
+    (property "JLC Rotation Offset" "270" (at 388.62 463.55 0)
+      (effects (font (size 1.27 1.27)) hide)
+    )
     (pin "1")
     (pin "2")
@@
       (effects (font (size 1.27 1.27)) hide)
     )
+    (property "JLC Rotation Offset" "270" (at 571.5 414.02 0)
+      (effects (font (size 1.27 1.27)) hide)
+    )
     (pin "1")
     (pin "2")
@@
       (effects (font (size 1.27 1.27)) hide)
     )
+    (property "JLC Rotation Offset" "270" (at 571.5 463.55 0)
+      (effects (font (size 1.27 1.27)) hide)
+    )
     (pin "1")
     (pin "2")
@@
       (effects (font (size 1.27 1.27)) hide)
     )
+    (property "JLC Rotation Offset" "270" (at 297.18 463.55 0)
+      (effects (font (size 1.27 1.27)) hide)
+    )
     (pin "1")
     (pin "2")
@@
       (effects (font (size 1.27 1.27)) hide)
     )
+    (property "JLC Rotation Offset" "180" (at 91.44 480.06 90)
+      (effects (font (size 1.27 1.27)) hide)
+    )
     (pin "1")
     (pin "2")
@@
       (effects (font (size 1.27 1.27)) hide)
     )
+    (property "JLC Rotation Offset" "270" (at 481.33 241.3 0)
+      (effects (font (size 1.27 1.27)) hide)
+    )
     (pin "1")
     (pin "2")
@@
       (effects (font (size 1.27 1.27)) hide)
     )
+    (property "JLC Rotation Offset" "270" (at 368.3 300.99 0)
+      (effects (font (size 1.27 1.27)) hide)
+    )
     (pin "1")
     (pin "2")
@@
       (effects (font (size 1.27 1.27)) hide)
     )
+    (property "JLC Rotation Offset" "180" (at 91.44 389.89 90)
+      (effects (font (size 1.27 1.27)) hide)
+    )
     (pin "1")
     (pin "2")
@@
       (effects (font (size 1.27 1.27)) hide)
     )
+    (property "JLC Rotation Offset" "270" (at 480.06 414.02 0)
+      (effects (font (size 1.27 1.27)) hide)
+    )
     (pin "1")
     (pin "2")
@@
       (effects (font (size 1.27 1.27)) hide)
     )
+    (property "JLC Rotation Offset" "270" (at 388.62 414.02 0)
+      (effects (font (size 1.27 1.27)) hide)
+    )
     (pin "1")
     (pin "2")
@@
       (effects (font (size 1.27 1.27)) hide)
     )
+    (property "JLC Rotation Offset" "270" (at 480.06 463.55 0)
+      (effects (font (size 1.27 1.27)) hide)
+    )
     (pin "1")
     (pin "2")
@@
       (effects (font (size 1.27 1.27)) hide)
     )
+    (property "JLC Rotation Offset" "270" (at 487.68 91.44 0)
+      (effects (font (size 1.27 1.27)) hide)
+    )
     (pin "1")
     (pin "2")
@@
       (effects (font (size 1.27 1.27)) hide)
     )
+    (property "JLC" "C213161" (at 237.49 304.8 0)
+      (effects (font (size 1.27 1.27)) hide)
+    )
+    (property "JLC Rotation Offset" "270" (at 237.49 304.8 0)
+      (effects (font (size 1.27 1.27)) hide)
+    )
     (pin "1")
     (pin "2")
@@
       (effects (font (size 1.27 1.27)) hide)
     )
+    (property "JLC Rotation Offset" "270" (at 368.3 241.3 0)
+      (effects (font (size 1.27 1.27)) hide)
+    )
     (pin "1")
     (pin "2")
@@
       (effects (font (size 1.27 1.27)) hide)
     )
+    (property "JLC Rotation Offset" "270" (at 448.31 91.44 0)
+      (effects (font (size 1.27 1.27)) hide)
+    )
     (pin "1")
     (pin "2")
@@
       (effects (font (size 1.27 1.27)) hide)
     )
+    (property "JLC Rotation Offset" "270" (at 191.77 461.01 0)
+      (effects (font (size 1.27 1.27)) hide)
+    )
     (pin "1")
     (pin "2")
@@
       (effects (font (size 1.27 1.27)) hide)
     )
+    (property "JLC" "C213161" (at 237.49 278.13 0)
+      (effects (font (size 1.27 1.27)) hide)
+    )
+    (property "JLC Rotation Offset" "270" (at 237.49 278.13 0)
+      (effects (font (size 1.27 1.27)) hide)
+    )
     (pin "1")
     (pin "2")
@@
       (effects (font (size 1.27 1.27)) hide)
     )
+    (property "JLC Rotation Offset" "270" (at 287.02 382.27 0)
+      (effects (font (size 1.27 1.27)) hide)
+    )
     (pin "1")
     (pin "2")
@@
       (effects (font (size 1.27 1.27)) hide)
     )
+    (property "JLC Rotation Offset" "270" (at 480.06 300.99 0)
+      (effects (font (size 1.27 1.27)) hide)
+    )
     (pin "1")
     (pin "2")
@@
       (effects (font (size 1.27 1.27)) hide)
     )
+    (property "JLC Rotation Offset" "270" (at 191.77 490.22 0)
+      (effects (font (size 1.27 1.27)) hide)
+    )
     (pin "1")
     (pin "2")
@@
       (effects (font (size 1.27 1.27)) hide)
     )
+    (property "JLC Rotation Offset" "270" (at 468.63 91.44 0)
+      (effects (font (size 1.27 1.27)) hide)
+    )
     (pin "1")
     (pin "2")
@@
       (effects (font (size 1.27 1.27)) hide)
     )
+    (property "JLC Rotation Offset" "180" (at 218.44 99.06 0)
+      (effects (font (size 1.27 1.27)) hide)
+    )
     (pin "1")
     (pin "2")
@@
       (effects (font (size 1.27 1.27)) hide)
     )
+    (property "JLC Rotation Offset" "270" (at 426.72 91.44 0)
+      (effects (font (size 1.27 1.27)) hide)
+    )
