File: hardware/surface-mount/europi-surface-mount.kicad_pcb (KiCad board)
At the start: 2 copper layers, 40.6 x 110 mm, 88 parts, among them J1 Conn_02x05_Odd_Even, J10 Output 6 Jack, J11 Conn_01x04_Pin, J2 Conn_01x04_Pin, J3 Output 1 Jack, J4 Output 4 Jack, J5 Analogue Input Jack, J6 Output 2 Jack, J7 Output 5 Jack, J8 Digital Input Jack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

Commit message: fix first revision issues
Connections:
- C15 pad 1: Net-(U5A-+) -> Net-(U5A--)
- R15 pad 2: Net-(U4C-+) -> Net-(U4C--)
- R18 pad 1: Net-(U4C-+) -> Net-(U4C--)
- R23 pad 2: Net-(U5A-+) -> Net-(U5A--)
- R28 pad 1: Net-(U5A-+) -> Net-(U5A--)
- U4 pad 10: Net-(U4C-+) -> GND
- U4 pad 9: GND -> Net-(U4C--)
- U5 pad 2: GND -> Net-(U5A--)
- U5 pad 3: Net-(U5A-+) -> GND
Routing:
- net Net-(U5A-+): track 25.1 -> 0.00 mm, vias 4 -> 0
- net Net-(U5A--): track 0.00 -> 19.7 mm, vias 0 -> 2
- net -12V: track 78.8 -> 88.1 mm
- net Net-(U4C-+): track 6.12 -> 0.00 mm
- net +12V: track 126.2 -> 131.4 mm, vias 7 -> 10
- net Net-(U4C--): track 0.00 -> 5.08 mm
- net GND: track 18.9 -> 14.0 mm, vias 11 -> 16
- net I2C_SDA: track 60.5 -> 62.6 mm, vias 1 -> 3
- net AIN_DETECT: track 40.6 -> 42.2 mm
- net ANALOGUE_IN: track 36.9 -> 38.4 mm
- net Net-(D3-K): track 33.8 -> 34.8 mm
- net +3.3V: track 129.4 -> 130.4 mm
- net I2C_SCL: track 63.0 -> 63.7 mm
- net OLED_SDA: track 58.6 -> 59.3 mm
- net OLED_SCL: track 65.9 -> 66.7 mm
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
Commit message: add version 1.1 number
Other:
- board text added: "v1.1"
Changed lines of the file:
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@@
+		)
+	)
+	(gr_text "v1.1"
+		(at 38.25 108.75 0)
+		(layer "B.SilkS")
+		(effects
+			(font
+				(size 1 1)
+				(thickness 0.2)
+				(bold yes)
+			)
+			(justify mirror)
 		)
 	)
