File: hardware/surface-mount/europi-surface-mount.kicad_pcb (KiCad board)
At the start: 2 copper layers, 40.6 x 110 mm, 91 parts, among them J1 Conn_02x05_Odd_Even, J10 Output 6 Jack, J11 Conn_01x04_Pin, J2 Conn_01x04_Pin, J3 Output 1 Jack, J4 Output 4 Jack, J5 Analogue Input Jack, J6 Output 2 Jack, J7 Output 5 Jack, J8 Digital Input Jack, J9 Output 3 Jack, Q1 2N2222, SW1 SW_Push, SW2 SW_Push, U2 PICO_RP2040, U3 TL074, U4 TL074, U5 MCP6002-xSN, U6 L7805

Commit message: Use JST port for I2C and add new JST port for I2S/Expander (#466)
* use JST port for I2C and add new JST port for I2S/Expander

* update build guide to match #466

* fix formatting of new rows

* fix photo for expansion headers
Parts:
- added J12: Conn_01x04_Pin, Connector_JST:JST_PH_B6B-PH-K_1x06_P2.00mm_Vertical, B.Cu at (3.05, 71.0)
- J11: footprint Connector_PinHeader_2.54mm:PinHeader_1x04_P2.54mm_Vertical -> Connector_JST:JST_PH_B4B-PH-K_1x04_P2.00mm_Vertical
- moved D2 14.0 mm to (14.0, 76.2)
- moved U6 2.06 mm to (12.7, 68.5)
- moved J11 1.91 mm to (3.09, 8.33), turned to 90 degrees
Connections:
- U2 pad 11: unconnected-(U2-GP8-Pad11) -> GP8
- U2 pad 12: unconnected-(U2-GP9-Pad12) -> GP9
- U2 pad 19: unconnected-(U2-GP14-Pad19) -> GP14
- U2 pad 20: unconnected-(U2-GP15-Pad20) -> GP15
Routing:
- net GP14: track 0.00 -> 61.9 mm, vias 0 -> 2
- net GP15: track 0.00 -> 56.0 mm, vias 0 -> 2
- net GP9: track 0.00 -> 50.4 mm, vias 0 -> 1
- net GP8: track 0.00 -> 49.6 mm, vias 0 -> 1
- net +3.3V: track 130.4 -> 154.2 mm, vias 7 -> 8
- net +5V: track 6.75 -> 25.2 mm, vias 0 -> 2
- net GND: track 13.4 -> 24.4 mm, vias 16 -> 27
- net OUT_1: track 43.5 -> 39.7 mm, vias 2 -> 3
- net OUT_4: track 53.0 -> 56.6 mm, vias 2 -> 3
- net +12V: track 131.6 -> 134.9 mm, vias 10 -> 8
- net Net-(D2-K): track 57.1 -> 54.1 mm
- net OUT_3: track 50.2 -> 52.8 mm, vias 2 -> 3
- net Net-(J3-T): track 67.4 -> 66.0 mm
- net Net-(J6-T): track 62.0 -> 63.4 mm
- net Net-(LED3-A): track 57.6 -> 56.4 mm
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Other:
- board text added: "14"
- board text added: "15"
- board text added: "8"
- board text added: "9"
- board text added: "REV4 23.04.2026"
- board text removed: "LICENSE: CERN OHL-S www.allensynthesis.co.uk"
- board text removed: "REV3 09.03.2026"

Commit message: increase led resistors to 5.1k to fix #479
Parts:
- R11, R12, R24, R25, R36, R37: value 4K7 -> 5K1
