File: hardware/surface-mount/europi-surface-mount.kicad_sch (KiCad schematic)
At the start: 90 parts, among them J1 Conn_02x05_Odd_Even, J10 Output 6 Jack, J11 Conn_01x04_Pin, J2 Conn_01x04_Pin, J3 Output 1 Jack, J4 Output 4 Jack, J5 Analogue Input Jack, J6 Output 2 Jack, J7 Output 5 Jack, J8 Digital Input Jack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

Commit message: add lcsc part number to d3
Parts:
- D3: LCSC Part (none) -> C5148475
Changed lines of the file:
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@@
+			)
+		)
+		(property "LCSC Part" "C5148475"
+			(at 276.86 187.96 0)
+			(effects
+				(font
+					(size 1.27 1.27)
+				)
+				(hide yes)
 			)
 		)
