File: hardware/surface-mount/europi-surface-mount.kicad_sch (KiCad schematic)
At the start: 88 parts, among them J1 Conn_02x05_Odd_Even, J10 Output 6 Jack, J11 Conn_01x04_Pin, J2 Conn_01x04_Pin, J3 Output 1 Jack, J4 Output 4 Jack, J5 Analogue Input Jack, J6 Output 2 Jack, J7 Output 5 Jack, J8 Digital Input Jack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

Commit message: fix first revision issues
Connections:
- net GND: now also U4.10 (+), U5.3 (+); no longer U4.9 (-), U5.2 (-)
- net at R15.2, R18.1: now also U4.9 (-); no longer U4.10 (+)
- net at C15.1, R23.2, R28.1: now also U5.2 (-); no longer U5.3 (+)
Changed lines of the file:
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@@
 		(lib_id "Amplifier_Operational:MCP6002-xSN")
 		(at 191.77 177.8 0)
-		(unit 1)
-		(exclude_from_sim no)
-		(in_bom yes)
-		(on_board yes)
-		(dnp no)
-		(fields_autoplaced yes)
+		(mirror x)
+		(unit 1)
+		(exclude_from_sim no)
+		(in_bom yes)
+		(on_board yes)
+		(dnp no)
 		(property "Reference" "U5"
-			(at 191.77 167.64 0)
+			(at 191.77 187.96 0)
 			(effects
 				(font
@@
 		)
 		(property "Value" "MCP6002-xSN"
-			(at 191.77 170.18 0)
+			(at 191.77 185.42 0)
 			(effects
 				(font
@@
 		(lib_id "Amplifier_Operational:TL074")
 		(at 156.21 175.26 0)
+		(mirror x)
 		(unit 3)
 		(exclude_from_sim no)
@@
 		(on_board yes)
 		(dnp no)
-		(fields_autoplaced yes)
 		(property "Reference" "U4"
-			(at 156.21 165.1 0)
+			(at 156.21 185.42 0)
 			(effects
 				(font
@@
 		)
 		(property "Value" "TL074"
-			(at 156.21 167.64 0)
+			(at 156.21 182.88 0)
 			(effects
 				(font
@@
 		)
 		(property "Footprint" "Package_SO:SOIC-14_3.9x8.7mm_P1.27mm"
-			(at 154.94 172.72 0)
+			(at 154.94 177.8 0)
 			(effects
 				(font
@@
 		)
 		(property "Datasheet" "http://www.ti.com/lit/ds/symlink/tl071.pdf"
-			(at 157.48 170.18 0)
-			(effects
-				(font
+			(at 157.48 180.34 0)
+			(effects
+				(font

Commit message: Minor surface-mount PCB changes (REV 3) (#458)
* add resistors to input detect and add oshwa cert mark

* add lcsc part number to d3
Parts:
- added R41, R42: 10K, Resistor_SMD:R_0603_1608Metric, symbol Device:R
- D3: LCSC Part (none) -> C5148475
Connections:
- net AIN_DETECT: now also R41.1; no longer J5.2 (TN)
- net DIN_DETECT: now also R42.1; no longer J8.2 (TN)
- new net: J8.2 (TN), R42.2
- new net: J5.2 (TN), R41.2
Changed lines of the file:
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@@
 	(wire
 		(pts
-			(xy 254 167.64) (xy 254 173.99)
+			(xy 254 166.37) (xy 254 173.99)
 		)
 		(stroke
@@
 	(wire
 		(pts
+			(xy 125.73 152.4) (xy 125.73 154.94)
+		)
+		(stroke
+			(width 0)
+			(type default)
+		)
+	)
+	(wire
+		(pts
 			(xy 134.62 74.93) (xy 134.62 69.85)
 		)
@@
 	(wire
 		(pts
+			(xy 254 156.21) (xy 254 158.75)
+		)
+		(stroke
+			(width 0)
+			(type default)
+		)
+	)
+	(wire
+		(pts
 			(xy 339.09 110.49) (xy 335.28 110.49)
 		)
@@
 	(global_label "AIN_DETECT"
 		(shape input)
-		(at 125.73 162.56 0)
+		(at 125.73 152.4 0)
 		(fields_autoplaced yes)
 		(effects
@@
 		)
 		(property "Intersheetrefs" "${INTERSHEET_REFS}"
-			(at 139.4799 162.56 0)
+			(at 139.4799 152.4 0)
 			(effects
 				(font
@@
 	(global_label "DIN_DETECT"
 		(shape input)
-		(at 254 167.64 0)
+		(at 254 156.21 0)
 		(fields_autoplaced yes)
 		(effects
@@
 		)
 		(property "Intersheetrefs" "${INTERSHEET_REFS}"
-			(at 267.9313 167.64 0)
+			(at 267.9313 156.21 0)
 			(effects
 				(font
@@
 	)
 	(symbol
+		(lib_id "Device:R")
+		(at 125.73 158.75 0)
+		(unit 1)
+		(exclude_from_sim no)
+		(in_bom yes)
+		(on_board yes)
+		(dnp no)
+		(property "Reference" "R41"
+			(at 127.508 157.5816 0)
+			(effects
+				(font
+					(size 1.27 1.27)
+				)
+				(justify left)
+			)
+		)
+		(property "Value" "10K"
+			(at 127.508 159.893 0)
+			(effects
+				(font
+					(size 1.27 1.27)
+				)
+				(justify left)
+			)
+		)
+		(property "Footprint" "Resistor_SMD:R_0603_1608Metric"
+			(at 123.952 158.75 90)
+			(effects
+				(font
+					(size 1.27 1.27)
+				)
+				(hide yes)
+			)
+		)
+		(property "Datasheet" "~"
+			(at 125.73 158.75 0)
+			(effects
+				(font
+					(size 1.27 1.27)
+				)
+				(hide yes)
+			)
+		)
+		(property "Description" ""
+			(at 125.73 158.75 0)
+			(effects
+				(font
+					(size 1.27 1.27)
+				)
+			)
+		)
+		(pin "1"
+		)
+		(pin "2"
+		)
+		(instances
+			(project "europi-surface-mount"
+				(path "/5701b80f-f006-4814-81c9-0c7f006088a9"
+					(reference "R41")
+					(unit 1)
+				)
+			)
+		)
+	)
+	(symbol
 		(lib_id "power:GND")
 		(at 328.93 189.23 270)
@@
 			)
 		)
+		(property "LCSC Part" "C5148475"
+			(at 276.86 187.96 0)
+			(effects
+				(font
+					(size 1.27 1.27)
+				)
+				(hide yes)
+			)
+		)
 		(pin "1"
 		)
@@
 					(unit 1)
 				)
+			)
+		)
+	)
+	(symbol
+		(lib_id "Device:R")
+		(at 254 162.56 0)
+		(unit 1)
+		(exclude_from_sim no)
+		(in_bom yes)
+		(on_board yes)
+		(dnp no)
+		(property "Reference" "R42"
+			(at 255.778 161.3916 0)
+			(effects
+				(font
+					(size 1.27 1.27)
+				)
+				(justify left)
+			)
+		)
+		(property "Value" "10K"
+			(at 255.778 163.703 0)
+			(effects
+				(font
+					(size 1.27 1.27)
+				)
+				(justify left)
+			)
+		)
+		(property "Footprint" "Resistor_SMD:R_0603_1608Metric"
+			(at 252.222 162.56 90)
+			(effects
+				(font
+					(size 1.27 1.27)
+				)
+				(hide yes)
+			)
+		)
+		(property "Datasheet" "~"
+			(at 254 162.56 0)
+			(effects
+				(font
+					(size 1.27 1.27)
+				)
+				(hide yes)
+			)
+		)
+		(property "Description" ""
+			(at 254 162.56 0)
+			(effects
+				(font
+					(size 1.27 1.27)
+				)
+			)
+		)
+		(pin "1"
+		)
+		(pin "2"
+		)
+		(instances
+			(project "europi-surface-mount"
+				(path "/5701b80f-f006-4814-81c9-0c7f006088a9"
+					(reference "R42")
+					(unit 1)
+				)
