File: hardware/surface-mount/europi-surface-mount.kicad_sch (KiCad schematic)
At the start: 90 parts, among them J1 Conn_02x05_Odd_Even, J10 Output 6 Jack, J11 Conn_01x04_Pin, J2 Conn_01x04_Pin, J3 Output 1 Jack, J4 Output 4 Jack, J5 Analogue Input Jack, J6 Output 2 Jack, J7 Output 5 Jack, J8 Digital Input Jack, J9 Output 3 Jack, Q1 2N2222, SW1 SW_Push, SW2 SW_Push, U2 PICO_RP2040, U3 TL074, U4 TL074, U5 MCP6002-xSN, U6 L7805

Commit message: Use JST port for I2C and add new JST port for I2S/Expander (#466)
* use JST port for I2C and add new JST port for I2S/Expander

* update build guide to match #466

* fix formatting of new rows

* fix photo for expansion headers
Parts:
- added J12: Conn_01x04_Pin, Connector_JST:JST_PH_B6B-PH-K_1x06_P2.00mm_Vertical, symbol Connector:Conn_01x06_Pin
- J11: footprint Connector_PinHeader_2.54mm:PinHeader_1x04_P2.54mm_Vertical -> Connector_JST:JST_PH_B4B-PH-K_1x04_P2.00mm_Vertical
Connections:
- net +3.3V: now also J12.2 (Pin_2)
- net GND: now also J12.1 (Pin_1)
- net GP8: now reaches U2.11 (GP8)
- net GP8: now also J12.6 (Pin_6)
- net GP9: now reaches U2.12 (GP9)
- net GP9: now also J12.5 (Pin_5)
- net GP14: now reaches U2.19 (GP14)
- net GP14: now also J12.4 (Pin_4)
- net GP15: now reaches U2.20 (GP15)
- net GP15: now also J12.3 (Pin_3)
- no-connect marks 23 -> 19
Other:
- note added: "I2S/Expander Port"

Commit message: increase led resistors to 5.1k to fix #479
Parts:
- R11, R12, R24, R25, R36, R37: value 4K7 -> 5K1
Changed lines of the file:
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@@
 			)
 		)
-		(property "Value" "4K7"
+		(property "Value" "5K1"
 			(at 157.8864 50.8 90)
 			(show_name no)
@@
 			)
 		)
-		(property "Value" "4K7"
+		(property "Value" "5K1"
 			(at 251.8664 50.8 90)
 			(show_name no)
@@
 			)
 		)
-		(property "Value" "4K7"
+		(property "Value" "5K1"
 			(at 347.1164 50.8 90)
 			(show_name no)
@@
 			)
 		)
-		(property "Value" "4K7"
+		(property "Value" "5K1"
 			(at 157.8864 106.68 90)
 			(show_name no)
@@
 			)
 		)
-		(property "Value" "4K7"
+		(property "Value" "5K1"
 			(at 251.8664 106.68 90)
 			(show_name no)
@@
 			)
 		)
-		(property "Value" "4K7"
+		(property "Value" "5K1"
 			(at 347.1164 106.68 90)
 			(show_name no)
